File: board/MystiqueJamma.brd (EAGLE design)
At the start: 120 x 145 mm, 75 parts, among them IC1 7805, IC2 74LS245N, IC4 74LS245N, IC5 CY7C1049CV33, IC6 TDA1543T

Commit message: included the FPGA board library
Parts:
- removed JP1, JP2: (no value), pinhead:2X20
- added U$1: C4E6-K"", FPGA-BOARD:E6V33
- moved R55 2.46 mm to (34.6, 68.8)
- moved R56 2.46 mm to (34.6, 71.9)
- moved R57 2.46 mm to (34.6, 75.0)
Connections:
- net +3V3: now also U$1.VCC1, U$1.VCC2; no longer JP1.2, JP2.1
- net GND: now also U$1.GND1, U$1.GND2, U$1.GND3, U$1.GND4; no longer JP1.23, JP1.24, JP2.23, JP2.24
- net SD_CS_144: now also U$1.I0_144; no longer JP2.33
- net SD_DATAIN_142: now also U$1.I0_142; no longer JP2.31
- net SD_DATAOUT_141: now also U$1.I0_141; no longer JP2.32
- net SD_SCLK_143: now also U$1.I0_143; no longer JP2.34
Changed lines of the file:
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@@
 </autorouter>
 <elements>
-<element name="JP1" library="pinhead" package="2X20" value="" x="110" y="111.1" rot="R90"/>
-<element name="JP2" library="pinhead" package="2X20" value="" x="56.6" y="111.1" rot="R90"/>
 <element name="IC1" library="SparkFun" package="TO220-IGO" value="7805" x="25.7" y="132.1" rot="R90"/>
 <element name="C1" library="rcl-2" package="E2,5-5" value="10uF" x="34.85" y="128.65" rot="R90"/>
@@
 <element name="R53" library="adafruit" package="0207/7" value="1k" x="93.125" y="65.857140625" rot="R180"/>
 <element name="R54" library="adafruit" package="0207/7" value="1k" x="93.125" y="62" rot="R180"/>
-<element name="R55" library="adafruit" package="0207/7" value="220" x="32.375" y="67.75" rot="R180"/>
-<element name="R56" library="adafruit" package="0207/7" value="220" x="32.375" y="70.875" rot="R180"/>
-<element name="R57" library="adafruit" package="0207/7" value="220" x="32.375" y="74" rot="R180"/>
+<element name="R55" library="adafruit" package="0207/7" value="220" x="34.625" y="68.75" rot="R180"/>
+<element name="R56" library="adafruit" package="0207/7" value="220" x="34.625" y="71.875" rot="R180"/>
+<element name="R57" library="adafruit" package="0207/7" value="220" x="34.625" y="75" rot="R180"/>
+<element name="U$1" library="FPGA-BOARD" package="E6V33" value="C4E6-K&quot;&quot;" x="53.5" y="159.75" rot="R270"/>
 </elements>
 <signals>
@@
 </signal>
 <signal name="GND">
-<contactref element="JP1" pad="23"/>
-<contactref element="JP1" pad="24"/>
-<contactref element="JP2" pad="23"/>
-<contactref element="JP2" pad="24"/>
 <contactref element="IC1" pad="GND"/>
 <contactref element="C1" pad="-"/>
@@
 <contactref element="R48" pad="2"/>
 <contactref element="JAMMA1" pad="14"/>
+<contactref element="U$1" pad="GND4"/>
+<contactref element="U$1" pad="GND3"/>
+<contactref element="U$1" pad="GND2"/>
+<contactref element="U$1" pad="GND1"/>
 <wire x1="5.5" y1="121.96" x2="5.5" y2="121.96" width="0" layer="19" extent="1-16"/>
 <wire x1="5.5" y1="118" x2="5.5" y2="121.96" width="0" layer="19" extent="1-1"/>
 <wire x1="5.5" y1="118" x2="5.5" y2="118" width="0" layer="19" extent="1-16"/>
 <wire x1="25.7" y1="132.1" x2="5.5" y2="121.96" width="0" layer="19" extent="1-1"/>
+<wire x1="54.9986" y1="113.0394" x2="50.56" y2="114" width="0" layer="19" extent="1-1"/>
 <wire x1="5.5" y1="86.32" x2="26.06" y2="79.75" width="0" layer="19" extent="16-16"/>
 <wire x1="5.5" y1="70.48" x2="5.5" y2="86.32" width="0" layer="19" extent="1-16"/>
@@
 <contactref element="U$2" pad="4"/>
 <contactref element="C5" pad="1"/>
-<contactref element="JP1" pad="2"/>
-<contactref element="JP2" pad="1"/>
 <contactref element="IC5" pad="9"/>
 <contactref element="IC5" pad="27"/>
 <contactref element="IC2" pad="20"/>
 <contactref element="IC4" pad="20"/>
-<wire x1="76.949" y1="118.865" x2="108.73" y2="86.97" width="0" layer="19" extent="1-1"/>
+<contactref element="U$1" pad="VCC2"/>
+<contactref element="U$1" pad="VCC1"/>
+<wire x1="76.949" y1="118.865" x2="114.7394" y2="85.0486" width="0" layer="19" extent="1-1"/>
 <wire x1="67.551" y1="120.135" x2="76.949" y2="118.865" width="0" layer="19" extent="1-1"/>
-<wire x1="57.87" y1="86.97" x2="67.551" y2="120.135" width="0" layer="19" extent="1-1"/>
-<wire x1="50.58" y1="49.59" x2="57.87" y2="86.97" width="0" layer="19" extent="1-1"/>
+<wire x1="57.5386" y1="85.0994" x2="67.551" y2="120.135" width="0" layer="19" extent="1-1"/>
+<wire x1="50.58" y1="49.59" x2="57.5386" y2="85.0994" width="0" layer="19" extent="1-1"/>
 <wire x1="46.66" y1="43.2999875" x2="50.58" y2="49.59" width="0" layer="19" extent="1-1"/>
 <wire x1="46.66" y1="39.41665625" x2="46.66" y2="43.2999875" width="0" layer="19" extent="1-1"/>
@@
 <signal name="SD_CS_144">
 <contactref element="U$2" pad="1"/>
-<contactref element="JP2" pad="33"/>
-<wire x1="93.1" y1="32.15" x2="57.87" y2="127.61" width="0" layer="19" extent="1-1"/>
+<contactref element="U$1" pad="I0_144"/>
+<wire x1="93.1" y1="32.15" x2="114.7394" y2="125.6886" width="0" layer="19" extent="1-1"/>
 </signal>
 <signal name="SD_SCLK_143">
 <contactref element="U$2" pad="5"/>
-<contactref element="JP2" pad="34"/>
-<wire x1="93.1" y1="22.15" x2="55.33" y2="127.61" width="0" layer="19" extent="1-1"/>
+<contactref element="U$1" pad="I0_143"/>
+<wire x1="93.1" y1="22.15" x2="117.2794" y2="125.6886" width="0" layer="19" extent="1-1"/>
 </signal>
 <signal name="SD_DATAIN_142">
 <contactref element="U$2" pad="2"/>
 <contactref element="R24" pad="1"/>
-<contactref element="JP2" pad="31"/>
-<wire x1="86.06" y1="29.75" x2="57.87" y2="125.07" width="0" layer="19" extent="1-1"/>
-<wire x1="93.1" y1="29.65" x2="86.06" y2="29.75" width="0" layer="19" extent="1-1"/>
+<contactref element="U$1" pad="I0_142"/>
+<wire x1="93.1" y1="29.65" x2="114.7394" y2="123.1486" width="0" layer="19" extent="1-1"/>
+<wire x1="86.06" y1="29.75" x2="93.1" y2="29.65" width="0" layer="19" extent="1-1"/>
 </signal>
 <signal name="SD_DATAOUT_141">
 <contactref element="U$2" pad="7"/>
 <contactref element="R23" pad="1"/>
-<contactref element="JP2" pad="32"/>
-<wire x1="86.06" y1="17.25" x2="55.33" y2="125.07" width="0" layer="19" extent="1-1"/>
-<wire x1="93.1" y1="17.15" x2="86.06" y2="17.25" width="0" layer="19" extent="1-1"/>
+<contactref element="U$1" pad="I0_141"/>
+<wire x1="93.1" y1="17.15" x2="117.2794" y2="123.1486" width="0" layer="19" extent="1-1"/>
+<wire x1="86.06" y1="17.25" x2="93.1" y2="17.15" width="0" layer="19" extent="1-1"/>
 </signal>
 <signal name="SRAM_A0">
@@
 <wire x1="74.4975" y1="65.857140625" x2="105.21" y2="64.079" width="0" layer="19" extent="1-1"/>
 <wire x1="74.4975" y1="73.571421875" x2="74.4975" y2="65.857140625" width="0" layer="19" extent="1-1"/>
-<wire x1="36.185" y1="74" x2="74.4975" y2="65.857140625" width="0" layer="19" extent="1-1"/>
+<wire x1="38.435" y1="75" x2="74.4975" y2="73.571421875" width="0" layer="19" extent="1-1"/>
 </signal>
 <signal name="VGA_GREEN">
@@
 <wire x1="85.935" y1="62" x2="105.21" y2="61.793" width="0" layer="19" extent="1-1"/>
 <wire x1="85.935" y1="73.571421875" x2="85.935" y2="62" width="0" layer="19" extent="1-1"/>
-<wire x1="36.185" y1="70.875" x2="85.935" y2="62" width="0" layer="19" extent="1-1"/>
+<wire x1="38.435" y1="71.875" x2="85.935" y2="73.571421875" width="0" layer="19" extent="1-1"/>
 </signal>
 <signal name="VGA_BLUE">
@@
 <wire x1="96.935" y1="62" x2="96.935" y2="73.571421875" width="0" layer="19" extent="1-1"/>
 <wire x1="105.21" y1="59.507" x2="96.935" y2="62" width="0" layer="19" extent="1-1"/>
-<wire x1="36.185" y1="67.75" x2="96.935" y2="62" width="0" layer="19" extent="1-1"/>
+<wire x1="38.435" y1="68.75" x2="96.935" y2="73.571421875" width="0" layer="19" extent="1-1"/>
 </signal>
 <signal name="N$4">
@@
 <contactref element="R36" pad="1"/>
 <contactref element="R37" pad="2"/>
-<contactref element="R37" pad="2"/>
 <wire x1="74.4975" y1="69.71428125" x2="74.4975" y2="81.285703125" width="0" layer="19" extent="1-1"/>
 <wire x1="66.8775" y1="62" x2="74.4975" y2="69.71428125" width="0" layer="19" extent="1-1"/>
@@
 <contactref element="R34" pad="1"/>
 <contactref element="R37" pad="1"/>
-<contactref element="R38" pad="2"/>
 <contactref element="R38" pad="2"/>
 <wire x1="66.8775" y1="65.857140625" x2="74.4975" y2="77.4285625" width="0" layer="19" extent="1-1"/>
@@
 <contactref element="R52" pad="2"/>
 <contactref element="R48" pad="1"/>
-<wire x1="96.935" y1="85.14284375" x2="89.315" y2="69.71428125" width="0" layer="19" extent="1-1"/>
-<wire x1="96.935" y1="88.999984375" x2="96.935" y2="85.14284375" width="0" layer="19" extent="1-1"/>
+<wire x1="96.935" y1="85.14284375" x2="96.935" y2="88.999984375" width="0" layer="19" extent="1-1"/>
+<wire x1="89.315" y1="69.71428125" x2="96.935" y2="85.14284375" width="0" layer="19" extent="1-1"/>
 </signal>
 <signal name="N$12">
@@
 <contactref element="R52" pad="1"/>
 <contactref element="R53" pad="2"/>
+<wire x1="96.935" y1="69.71428125" x2="96.935" y2="81.285703125" width="0" layer="19" extent="1-1"/>
 <wire x1="89.315" y1="65.857140625" x2="96.935" y2="69.71428125" width="0" layer="19" extent="1-1"/>
-<wire x1="96.935" y1="81.285703125" x2="96.935" y2="69.71428125" width="0" layer="19" extent="1-1"/>
 </signal>
 <signal name="N$13">
@@
 <contactref element="R53" pad="1"/>
 <contactref element="R54" pad="2"/>
+<wire x1="96.935" y1="65.857140625" x2="96.935" y2="77.4285625" width="0" layer="19" extent="1-1"/>
 <wire x1="89.315" y1="62" x2="96.935" y2="65.857140625" width="0" layer="19" extent="1-1"/>
-<wire x1="96.935" y1="77.4285625" x2="96.935" y2="65.857140625" width="0" layer="19" extent="1-1"/>
 </signal>
 <signal name="VGA_B0">
@@
 <contactref element="JAMMA1" pad="12"/>
 <contactref element="R57" pad="2"/>
-<wire x1="28.565" y1="74" x2="5.5" y2="78.4" width="0" layer="19" extent="1-1"/>
+<wire x1="5.5" y1="78.4" x2="30.815" y2="75" width="0" layer="19" extent="1-1"/>
 </signal>
 <signal name="JVIDEO_BLUE">
 <contactref element="JAMMA1" pad="13"/>
 <contactref element="R55" pad="2"/>
-<wire x1="28.565" y1="67.75" x2="5.5" y2="74.44" width="0" layer="19" extent="1-1"/>
+<wire x1="5.5" y1="74.44" x2="30.815" y2="68.75" width="0" layer="19" extent="1-1"/>
 </signal>
 <signal name="JVIDEO_GREEN">
 <contactref element="JAMMA2" pad="N"/>
 <contactref element="R56" pad="2"/>
-<wire x1="28.565" y1="70.875" x2="5.5" y2="78.4" width="0" layer="19" extent="16-16"/>
+<wire x1="5.5" y1="78.4" x2="30.815" y2="71.875" width="0" layer="19" extent="16-16"/>
 </signal>
 <signal name="VGA_HSYNC">

Commit message: docs
Parts:
- removed U$1: C4E6-K"", FPGA-BOARD:E6V33
- added B1: (no value), FPGA-BOARD:E6V33
- moved C3 3.18 mm to (44.5, 102.5)
- moved R25 3.18 mm to (44.5, 111.8)
- moved R26 3.18 mm to (44.5, 107.5)
- moved R27 3.18 mm to (44.5, 116.0)
Connections:
- net +3V3: now also B1.VCC1, B1.VCC2, B1.VCC3; no longer U$1.VCC1, U$1.VCC2
- net GND: now also B1.GND1, B1.GND2, B1.GND3, B1.GND4; no longer U$1.GND1, U$1.GND2, U$1.GND3, U$1.GND4
- net SD_CS_144: now also B1.I0_144; no longer U$1.I0_144
- net SD_DATAIN_142: now also B1.I0_142; no longer U$1.I0_142
- net SD_DATAOUT_141: now also B1.I0_141; no longer U$1.I0_141
- net SD_SCLK_143: now also B1.I0_143; no longer U$1.I0_143
Changed lines of the file:
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@@
 <element name="IC5" library="memory-sram" package="SOJV36-400" value="CY7C1049CV33" x="72.25" y="119.5" rot="R270"/>
 <element name="IC6" library="TDA1543" package="SOIC-16NW" value="TDA1543T" x="31.25" y="108" rot="R270"/>
-<element name="R25" library="adafruit" package="0207/7" value="1k" x="46.75" y="114" rot="R180"/>
-<element name="R26" library="adafruit" package="0207/7" value="2k" x="46.75" y="109.75" rot="R180"/>
-<element name="C3" library="adafruit" package="C025-025X050" value="100nF" x="46.75" y="104.75"/>
-<element name="R27" library="adafruit" package="0207/7" value="2k" x="46.75" y="118.25" rot="R180"/>
+<element name="R25" library="adafruit" package="0207/7" value="1k" x="44.5" y="111.75" rot="R180"/>
+<element name="R26" library="adafruit" package="0207/7" value="2k" x="44.5" y="107.5" rot="R180"/>
+<element name="C3" library="adafruit" package="C025-025X050" value="100nF" x="44.5" y="102.5"/>
+<element name="R27" library="adafruit" package="0207/7" value="2k" x="44.5" y="116" rot="R180"/>
 <element name="C4" library="adafruit" package="E5-6" value="4.7uF" x="34.875" y="89" rot="R180"/>
 <element name="C6" library="adafruit" package="E5-6" value="4.7uF" x="34.875" y="81.5" rot="R180"/>
@@
 <element name="R56" library="adafruit" package="0207/7" value="220" x="34.625" y="71.875" rot="R180"/>
 <element name="R57" library="adafruit" package="0207/7" value="220" x="34.625" y="75" rot="R180"/>
-<element name="U$1" library="FPGA-BOARD" package="E6V33" value="C4E6-K&quot;&quot;" x="53.5" y="159.75" rot="R270"/>
+<element name="B1" library="FPGA-BOARD" package="E6V33" value="" x="84.75" y="160.75" rot="MR270"/>
 </elements>
 <signals>
@@
 <contactref element="R48" pad="2"/>
 <contactref element="JAMMA1" pad="14"/>
-<contactref element="U$1" pad="GND4"/>
-<contactref element="U$1" pad="GND3"/>
-<contactref element="U$1" pad="GND2"/>
-<contactref element="U$1" pad="GND1"/>
+<contactref element="B1" pad="GND3"/>
+<contactref element="B1" pad="GND4"/>
+<contactref element="B1" pad="GND1"/>
+<contactref element="B1" pad="GND2"/>
+<wire x1="113.3504" y1="113.76" x2="115.8904" y2="113.76" width="0" layer="19" extent="1-1"/>
+<wire x1="89.315" y1="85.14284375" x2="113.3504" y2="113.76" width="0" layer="19" extent="1-1"/>
+<wire x1="78.315" y1="85.14284375" x2="89.315" y2="85.14284375" width="0" layer="19" extent="1-1"/>
+<wire x1="66.8775" y1="85.14284375" x2="78.315" y2="85.14284375" width="0" layer="19" extent="1-1"/>
+<wire x1="45.77" y1="102.5" x2="66.8775" y2="85.14284375" width="0" layer="19" extent="1-1"/>
+<wire x1="48.31" y1="107.5" x2="45.77" y2="102.5" width="0" layer="19" extent="1-1"/>
+<wire x1="48.31" y1="111.75" x2="48.31" y2="107.5" width="0" layer="19" extent="1-1"/>
+<wire x1="48.31" y1="116" x2="48.31" y2="111.75" width="0" layer="19" extent="1-1"/>
+<wire x1="53.6096" y1="113.7092" x2="48.31" y2="107.5" width="0" layer="19" extent="1-1"/>
+<wire x1="56.1496" y1="113.7092" x2="53.6096" y2="113.7092" width="0" layer="19" extent="1-1"/>
+<wire x1="67.551" y1="118.865" x2="56.1496" y2="113.7092" width="0" layer="19" extent="1-1"/>
+<wire x1="76.949" y1="120.135" x2="67.551" y2="118.865" width="0" layer="19" extent="1-1"/>
+<wire x1="34.85" y1="129.92" x2="48.31" y2="116" width="0" layer="19" extent="1-1"/>
+<wire x1="34.85" y1="134.98" x2="34.85" y2="129.92" width="0" layer="19" extent="1-1"/>
+<wire x1="25.7" y1="132.1" x2="34.85" y2="129.92" width="0" layer="19" extent="1-1"/>
+<wire x1="26.835" y1="106.095" x2="45.77" y2="102.5" width="0" layer="19" extent="1-1"/>
+<wire x1="5.5" y1="121.96" x2="25.7" y2="132.1" width="0" layer="19" extent="1-1"/>
 <wire x1="5.5" y1="121.96" x2="5.5" y2="121.96" width="0" layer="19" extent="1-16"/>
 <wire x1="5.5" y1="118" x2="5.5" y2="121.96" width="0" layer="19" extent="1-1"/>
 <wire x1="5.5" y1="118" x2="5.5" y2="118" width="0" layer="19" extent="1-16"/>
-<wire x1="25.7" y1="132.1" x2="5.5" y2="121.96" width="0" layer="19" extent="1-1"/>
-<wire x1="54.9986" y1="113.0394" x2="50.56" y2="114" width="0" layer="19" extent="1-1"/>
+<wire x1="26.06" y1="79.75" x2="26.835" y2="106.095" width="0" layer="19" extent="1-1"/>
 <wire x1="5.5" y1="86.32" x2="26.06" y2="79.75" width="0" layer="19" extent="16-16"/>
 <wire x1="5.5" y1="70.48" x2="5.5" y2="86.32" width="0" layer="19" extent="1-16"/>
+<wire x1="27.72" y1="57.21" x2="26.06" y2="79.75" width="0" layer="19" extent="1-1"/>
+<wire x1="48.04" y1="49.59" x2="27.72" y2="57.21" width="0" layer="19" extent="1-1"/>
+<wire x1="50.58" y1="57.21" x2="48.04" y2="49.59" width="0" layer="19" extent="1-1"/>
+<wire x1="54.69" y1="29.58" x2="48.04" y2="49.59" width="0" layer="19" extent="1-1"/>
+<wire x1="62.31" y1="27.04" x2="54.69" y2="29.58" width="0" layer="19" extent="1-1"/>
+<wire x1="82.25" y1="26.77" x2="62.31" y2="27.04" width="0" layer="19" extent="1-1"/>
+<wire x1="93.1" y1="27.15" x2="82.25" y2="26.77" width="0" layer="19" extent="1-1"/>
+<wire x1="93.1" y1="19.65" x2="93.1" y2="27.15" width="0" layer="19" extent="1-1"/>
+<wire x1="54.69" y1="6.72" x2="62.31" y2="27.04" width="0" layer="19" extent="1-1"/>
+<wire x1="115.8" y1="11.45" x2="93.1" y2="19.65" width="0" layer="19" extent="1-1"/>
+<wire x1="105.21" y1="54.935" x2="93.1" y2="27.15" width="0" layer="19" extent="1-1"/>
+<wire x1="107.75" y1="56.078" x2="105.21" y2="54.935" width="0" layer="19" extent="1-1"/>
 <wire x1="5.5" y1="19" x2="27.72" y2="57.21" width="0" layer="19" extent="16-16"/>
 <wire x1="5.5" y1="19" x2="5.5" y2="19" width="0" layer="19" extent="1-16"/>
@@
 <wire x1="25.7" y1="134.64" x2="34.85" y2="137.52" width="0" layer="19" extent="1-1"/>
 <wire x1="35.665" y1="106.095" x2="25.7" y2="134.64" width="0" layer="19" extent="1-1"/>
-<wire x1="45.48" y1="104.75" x2="35.665" y2="106.095" width="0" layer="19" extent="1-1"/>
+<wire x1="43.23" y1="102.5" x2="35.665" y2="106.095" width="0" layer="19" extent="1-1"/>
 </signal>
 <signal name="+3V3">
@@
 <contactref element="IC2" pad="20"/>
 <contactref element="IC4" pad="20"/>
-<contactref element="U$1" pad="VCC2"/>
-<contactref element="U$1" pad="VCC1"/>
-<wire x1="76.949" y1="118.865" x2="114.7394" y2="85.0486" width="0" layer="19" extent="1-1"/>
+<contactref element="B1" pad="VCC2"/>
+<contactref element="B1" pad="VCC3"/>
+<contactref element="B1" pad="VCC1"/>
+<wire x1="76.949" y1="118.865" x2="113.3504" y2="85.82" width="0" layer="19" extent="1-1"/>
 <wire x1="67.551" y1="120.135" x2="76.949" y2="118.865" width="0" layer="19" extent="1-1"/>
-<wire x1="57.5386" y1="85.0994" x2="67.551" y2="120.135" width="0" layer="19" extent="1-1"/>
-<wire x1="50.58" y1="49.59" x2="57.5386" y2="85.0994" width="0" layer="19" extent="1-1"/>
+<wire x1="56.1496" y1="85.7692" x2="67.551" y2="120.135" width="0" layer="19" extent="1-1"/>
+<wire x1="53.6096" y1="85.7692" x2="56.1496" y2="85.7692" width="0" layer="19" extent="1-1"/>
+<wire x1="50.58" y1="49.59" x2="53.6096" y2="85.7692" width="0" layer="19" extent="1-1"/>
 <wire x1="46.66" y1="43.2999875" x2="50.58" y2="49.59" width="0" layer="19" extent="1-1"/>
 <wire x1="46.66" y1="39.41665625" x2="46.66" y2="43.2999875" width="0" layer="19" extent="1-1"/>
@@
 <signal name="SD_CS_144">
 <contactref element="U$2" pad="1"/>
-<contactref element="U$1" pad="I0_144"/>
-<wire x1="93.1" y1="32.15" x2="114.7394" y2="125.6886" width="0" layer="19" extent="1-1"/>
+<contactref element="B1" pad="I0_144"/>
+<wire x1="93.1" y1="32.15" x2="56.1496" y2="126.4092" width="0" layer="19" extent="1-1"/>
 </signal>
 <signal name="SD_SCLK_143">
 <contactref element="U$2" pad="5"/>
-<contactref element="U$1" pad="I0_143"/>
-<wire x1="93.1" y1="22.15" x2="117.2794" y2="125.6886" width="0" layer="19" extent="1-1"/>
+<contactref element="B1" pad="I0_143"/>
+<wire x1="93.1" y1="22.15" x2="53.6096" y2="126.4092" width="0" layer="19" extent="1-1"/>
 </signal>
 <signal name="SD_DATAIN_142">
 <contactref element="U$2" pad="2"/>
 <contactref element="R24" pad="1"/>
-<contactref element="U$1" pad="I0_142"/>
-<wire x1="93.1" y1="29.65" x2="114.7394" y2="123.1486" width="0" layer="19" extent="1-1"/>
-<wire x1="86.06" y1="29.75" x2="93.1" y2="29.65" width="0" layer="19" extent="1-1"/>
+<contactref element="B1" pad="I0_142"/>
+<wire x1="86.06" y1="29.75" x2="56.1496" y2="123.8692" width="0" layer="19" extent="1-1"/>
+<wire x1="93.1" y1="29.65" x2="86.06" y2="29.75" width="0" layer="19" extent="1-1"/>
 </signal>
 <signal name="SD_DATAOUT_141">
 <contactref element="U$2" pad="7"/>
 <contactref element="R23" pad="1"/>
-<contactref element="U$1" pad="I0_141"/>
-<wire x1="93.1" y1="17.15" x2="117.2794" y2="123.1486" width="0" layer="19" extent="1-1"/>
-<wire x1="86.06" y1="17.25" x2="93.1" y2="17.15" width="0" layer="19" extent="1-1"/>
+<contactref element="B1" pad="I0_141"/>
+<wire x1="86.06" y1="17.25" x2="53.6096" y2="123.8692" width="0" layer="19" extent="1-1"/>
+<wire x1="93.1" y1="17.15" x2="86.06" y2="17.25" width="0" layer="19" extent="1-1"/>
 </signal>
 <signal name="SRAM_A0">
@@
 <contactref element="IC6" pad="13"/>
 <contactref element="R25" pad="2"/>
-<wire x1="35.665" y1="108.635" x2="42.94" y2="114" width="0" layer="19" extent="1-1"/>
+<wire x1="35.665" y1="108.635" x2="40.69" y2="111.75" width="0" layer="19" extent="1-1"/>
 </signal>
 <signal name="L_A">
@@
 <contactref element="IC6" pad="12"/>
 <contactref element="C6" pad="+"/>
-<wire x1="35.665" y1="107.365" x2="42.94" y2="109.75" width="0" layer="19" extent="1-1"/>
+<wire x1="35.665" y1="107.365" x2="40.69" y2="107.5" width="0" layer="19" extent="1-1"/>
 <wire x1="37.415" y1="81.5" x2="35.665" y2="107.365" width="0" layer="19" extent="1-1"/>
 </signal>
@@
 <contactref element="R27" pad="2"/>
 <contactref element="C4" pad="+"/>
-<wire x1="35.665" y1="109.905" x2="42.94" y2="118.25" width="0" layer="19" extent="1-1"/>
+<wire x1="35.665" y1="109.905" x2="40.69" y2="116" width="0" layer="19" extent="1-1"/>
 <wire x1="37.415" y1="89" x2="35.665" y2="109.905" width="0" layer="19" extent="1-1"/>
 </signal>
