File: board/eagle/MystiqueJamma.brd (EAGLE design)
At the start: 120 x 145 mm, 74 parts, among them IC1 7805, IC2 74LS245N, IC4 74LS245N, IC5 CY7C1049CV33, IC6 TDA1543T

Commit message: Shift registers to read controllers, new libs
Parts:
- removed B1: (no value), FPGA-BOARD:E6V33
- removed JAMMA1: JAMMA_TOP, JAMMA:JAMMA_TOP
- removed JAMMA2: JAMMA_BOTTOM, JAMMA:JAMMA_BOTTOM
- removed X1: (no value), adafruit:HDF15H
- added C10, C8, C9: 10uF, rcl-2:E2,5-5
- added C11, C12, C13, C14, C15, C16, C17, C18, C19, C20, C21, C27, C28, C29, C7: 100nF, adafruit:C1206
- added C22, C25, C26: (no value), rcl:E2-4
- added C23: 100u/25V, rcl:E3,5-8
- added C24: 1000u/25V, rcl:E3,5-8
- added D2, D3: (no value), diode:SOD80C
- added IC10: TDA2030V, linear:CB360
- added IC11: LA4425V, LA4425:LA4425
- added IC3, IC7: 74LS245DW, 74xx-us:SO20W
- added IC8: (no value), TLS1233:DIL20
- added IC9: 74HC4021D, 40xx:SO16
- added K1: JAMMA-EDGE, JAMMA:JAMMA-EDGE
- added R58: (no value), pot:SP19L
- added R59, R60, R61, R62, R63, R64, R65, R66, R67, R68, R69, R70, R71, R72, R73, R74, R75, R76, R77, R78, R79, R80, R81, R82, R83, R84, R85, R86, R87, R88, R89, R90, R91, R92, R93: 330, adafruit:M1206
- added U$3: (no value), FPGA-BOARD:E6V33
- added X2: 1503_09, con-lumberg:1503_09
- added X4: (no value), con-subd:HDF15H
- C1: value 10uF -> 100uF
- C3: device adafruit:C025-025X050 -> adafruit:C1206
- C5: device adafruit:C025-024X044 -> adafruit:C1206
- IC2, IC4: value 74LS245N -> 74HC4021D; device 74xx-us:DIL20 -> 40xx:SO16
- R1, R3, R5: value 330 -> 470; device adafruit:0207/7 -> adafruit:R1206
- R10, R12, R14, R16, R18, R20, R22, R8: value 10k -> 330; device adafruit:0207/7 -> adafruit:M1206
- R11, R13, R15, R17, R19, R21, R29, R7: device adafruit:0207/7 -> adafruit:M1206
- R2, R4, R6: value 10k -> 470; device adafruit:0207/7 -> adafruit:R1206
- R23, R24, R25, R26, R27, R28: device adafruit:0207/7 -> adafruit:R1206
- R30: value 20k -> 330; device adafruit:0207/7 -> adafruit:M1206
- R31, R32, R33, R34, R35, R39, R40, R41, R42, R43, R47, R48, R49, R50, R51: value 2k -> 330; device adafruit:0207/7 -> adafruit:M1206
- R36, R37, R38, R44, R45, R46, R52, R53, R54: value 1k -> 330; device adafruit:0207/7 -> adafruit:M1206
- R55, R56: value 220 -> 330; device adafruit:0207/7 -> adafruit:M1206
- R57: value 220 -> (none); device adafruit:0207/7 -> pot:SP19L
- R9: value 330 -> (none); device adafruit:0207/7 -> pot:3RP/1610N
- moved R6 1077.6 mm to (-181.6, -1018.5)
- moved R5 1069.3 mm to (-181.6, -1012.2), turned to 0 degrees
- moved R4 1069.1 mm to (-181.6, -1005.8)
- moved R3 1060.8 mm to (-181.6, -999.5), turned to 0 degrees
- moved R1 1058.4 mm to (-181.6, -993.1), turned to 0 degrees
- moved R56 1055.6 mm to (-181.6, -961.4), turned to 0 degrees
- moved R54 1047.4 mm to (-181.6, -948.7), turned to 0 degrees
- moved R55 1046.4 mm to (-181.6, -955.0), turned to 0 degrees
- moved R53 1045.0 mm to (-181.6, -942.3), turned to 0 degrees
- moved R52 1042.6 mm to (-181.6, -936.0), turned to 0 degrees
- moved R51 1040.2 mm to (-181.6, -929.6), turned to 0 degrees
- moved R48 1032.9 mm to (-181.6, -910.6), turned to 0 degrees
- moved R49 1027.9 mm to (-176.5, -910.6), turned to 0 degrees
- moved R39 1009.3 mm to (-181.6, -885.2), turned to 0 degrees
- moved R41 1007.9 mm to (-181.6, -891.5), turned to 0 degrees
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Connections:
- net DAC_DATA renamed I2S_DATA
- net DAC_FSYNC renamed IS2_WS
- net DAC_SCK renamed I2S_BCK
- net P1B5_3V renamed N$43
- net P1S_3V renamed CNTR_DAT
- removed net +12: D1.A, JAMMA1.6
- removed net +5REG: C2.+, C3.1, IC1.OUT, IC6.11
- removed net 12+: JAMMA2.F
- removed net CS1_: IC2.18, R1.1, R2.1
- removed net CS1_3V: IC2.2
- removed net JVIDEO_BLUE: JAMMA1.13, R55.2
- removed net JVIDEO_GREEN: JAMMA2.N, R56.2
- removed net JVIDEO_RED: JAMMA1.12, R57.2
- removed net P1B1_: IC2.12, R15.1, R16.1
- removed net P1B1_3V: IC2.8
- removed net P1B2_: IC2.11, R17.1, R18.1
- removed net P1B2_3V: IC2.9
- removed net P1B3_: IC4.18, R19.1, R20.1
- removed net P1B3_3V: IC4.2
- removed net P1B4_: IC4.17, R21.1, R22.1
- removed net P1B4_3V: IC4.3
- removed net P1B5_: IC4.16, R13.1, R14.1
- removed net P1D_: IC2.15, R7.1, R8.1
- removed net P1D_3V: IC2.5
- removed net P1L_: IC2.14, R10.1, R9.1
- removed net P1L_3V: IC2.6
- removed net P1R_: IC2.13, R11.1, R12.1
- removed net P1R_3V: IC2.7
- removed net P1S_: IC2.17, R3.1, R4.1
- removed net P1U_: IC2.16, R5.1, R6.1
- removed net P1U_3V: IC2.4
- removed net SD_CS_144: B1.I0_144, U$2.1
- removed net SD_DATAIN_142: B1.I0_142, R24.1, U$2.2
- removed net SD_DATAOUT_141: B1.I0_141, R23.1, U$2.7
- removed net SD_SCLK_143: B1.I0_143, U$2.5
- removed net VGA_B0: R47.2
- removed net VGA_B1: R49.2
- removed net VGA_B2: R50.2
- removed net VGA_B3: R51.2
- removed net VGA_BLUE: R51.1, R54.1, R55.1, X1.3
- removed net VGA_G0: R39.2
- removed net VGA_G1: R41.2
- removed net VGA_G2: R42.2
- removed net VGA_G3: R43.2
- removed net VGA_GREEN: R43.1, R46.1, R56.1, X1.2
- removed net VGA_HSYNC: JAMMA2.P, X1.13
- removed net VGA_R0: R31.2
- removed net VGA_R1: R33.2
- removed net VGA_R2: R34.2
- removed net VGA_R3: R35.2
- removed net VGA_RED: R35.1, R38.1, R57.1, X1.1
- removed net VGA_VSYNC: X1.14
- new net +12V: C23.+, C27.1, D1.A, D3.C, IC10.5, IC11.5, IC8.16, IC8.2, K1.6, K1.F, R2.1, R53.2, R54.2, R55.2
- new net B0: IC7.2
- new net B1: IC7.3
- new net B2: IC7.4
- new net B3: IC7.5
- new net BURST_GATE: IC8.11
- new net CNTR_CLK: IC2.10, IC4.10, IC9.10
- new net CNTR_LATCH: IC2.9, IC4.9, IC9.9
- new net CSY: IC7.8
- new net G0: IC3.6
- new net G1: IC3.7
- new net G2: IC3.8
- new net G3: IC3.9
- new net GATE: IC7.9
- new net HSY: IC7.6
- new net JAMMA-BLUE: K1.13, R52.2
- new net JAMMA-CSYNC: K1.P
- new net JAMMA-GREEN: K1.N, R51.2
- new net JAMMA-RED: K1.12, R50.2
- new net JAMMA_AUDIO: R28.2, R29.2, R9.3
- new net LAA: R29.1, X2.4
- new net N$14: IC7.18
- new net N$15: IC7.16
- new net N$16: IC7.15
- new net N$17: IC7.14
- new net N$18: IC7.13
- new net N$19: IC7.12
- new net N$20: IC7.11
- new net N$21: C16.1, IC8.1, IC8.19, IC8.20, R58.S
- new net N$22: C11.1, IC8.4
- new net N$23: C12.1, IC8.7
- new net N$24: C13.1, IC8.9
- new net N$25: IC8.18, R50.1, R59.2
- new net N$26: IC8.15, R51.1, R60.2, R61.2
- new net N$27: IC8.13, R52.1
- new net N$28: C14.1, IC8.10, R57.S
- new net N$29: R53.1, R57.E
- new net N$30: IC2.7, R63.1
- new net N$31: R55.1, R58.E
- new net N$32: IC2.6, R7.1
- new net N$33: IC2.5, R8.1
- new net N$34: C15.1, IC8.12, IC8.14, IC8.17, R54.1, R56.2
- new net N$35: IC2.4, R10.1
- new net N$36: IC2.13, R11.1
- new net N$37: IC2.14, R12.1
- new net N$38: IC2.15, R13.1
- new net N$39: IC2.1, R14.1
- new net N$40: IC4.7
- new net N$41: IC4.6
- new net N$42: IC4.5
- new net N$44: IC4.13
- new net N$45: C22.+, R1.1, R2.2, R3.1
- new net N$46: R7.2
- new net N$47: R63.2
- new net N$48: IC4.14
- new net N$49: IC4.15
- new net N$50: IC4.1
- new net N$51: IC9.7
- new net N$52: IC9.6
- new net N$53: IC9.5
- new net N$54: IC9.4
- new net N$55: IC9.13
- new net N$56: IC9.14
- new net N$57: IC9.15
- new net N$58: IC9.1
- new net N$59: C28.1, R6.2
- new net N$60: C26.+, R4.2
- new net N$61: R8.2
- new net N$62: R10.2
- new net N$63: R12.2
- new net N$64: R11.2
- new net N$65: R13.2
- new net N$66: R14.2
- new net N$71: IC10.2, R4.1, R5.2
- new net N$88: IC2.11, IC4.3
- new net N$89: IC4.11, IC9.3
- new net N$91: C25.-, R9.2
- new net N$92: C25.+, IC10.1, IC11.1, R3.2
- new net N$93: C24.+, D2.C, D3.A, IC10.4, IC11.4, R5.1, R6.1
- new net R0: IC3.2
- new net R1: IC3.3
- new net R2: IC3.4
- new net R3: IC3.5
- new net RAA: R28.1, X2.5
- new net SD_CS: U$2.1
- new net SD_DATAIN: R24.1, U$2.2
- new net SD_DATAOUT: R23.1, U$2.7
- new net SD_SCLK: U$2.5
- new net VGA-BLUE: C10.-, R35.2, X4.3
- new net VGA-GREEN: C9.-, R36.2, X4.2
- new net VGA-HSYNC: X4.13
- new net VGA-RED: C8.-, R31.2, R32.2, R33.2, R34.2, R47.2, X4.1
- new net VGA-VSYNC: X4.14
- new net VGA_DETECT: X4.5
- new net VSY: IC7.7
- net +3V3: now also C19.1, C20.1, C21.1, IC2.16, IC4.16, IC9.16, R70.2, R71.2, R72.2, R73.2, R74.2, R75.2, R76.2, R77.2, R78.2, R79.2, R80.2, R81.2, R82.2, R83.2, R84.2, R85.2, R86.2, R87.2, R88.2, R89.2, R90.2, R91.2, R92.2, R93.2, U$3.VCC1, U$3.VCC2, U$3.VCC3; no longer B1.VCC1, B1.VCC2, B1.VCC3, IC2.20, IC4.20, R10.2, R12.2, R14.2, R16.2, R18.2, R2.2, R20.2, R22.2, R4.2, R6.2, R8.2
- net +5V: now also C17.1, C18.1, C2.+, C3.1, C7.1, IC1.OUT, IC3.20, IC6.11, IC7.20, K1.3, K1.4, K1.C, K1.D; no longer JAMMA1.3, JAMMA1.4, JAMMA2.C, JAMMA2.D
- net -5V: now also K1.5, K1.E; no longer JAMMA1.5, JAMMA2.E
- net COINSW1: now also K1.16; no longer JAMMA1.16, R1.2
- net GND: now also C11.2, C12.2, C13.2, C14.2, C15.2, C16.2, C17.2, C18.2, C19.2, C20.2, C21.2, C22.-, C23.-, C26.-, C27.2, C28.2, C29.2, C7.2, D2.A, IC10.3, IC11.2, IC11.3, IC2.8, IC3.10, IC3.19, IC4.8, IC7.10, IC7.19, IC8.6, IC9.11, IC9.8, K1.#E, K1.#F, K1.1, K1.14, K1.2, K1.27, K1.28, K1.A, K1.B, K1.L, R1.2, R35.1, R36.1, R47.1, R56.1, R57.A, R58.A, R59.1, R60.1, R61.1, R9.1, U$3.GND1, U$3.GND2, U$3.GND3, U$3.GND4, X2.1, X4.10, X4.6, X4.7, X4.8; no longer B1.GND1, B1.GND2, B1.GND3, B1.GND4, IC2.1, IC2.10, IC2.19, IC4.1, IC4.10, IC4.19, JAMMA1.1, JAMMA1.14, JAMMA1.2, JAMMA1.27, JAMMA1.28, JAMMA2.A, JAMMA2.B, JAMMA2.L, JAMMA2._E, JAMMA2._F, R30.1, R32.2, R40.2, R48.2, X1.10, X1.5
- net JAMMA_SPK+: now also C24.-, K1.10; no longer JAMMA1.10, R28.2, R29.2, R30.2
- net L_AUDIO: now also X2.2; no longer R29.1
- net N$1: now also IC3.17; no longer R31.1, R36.2
- net N$10: now also IC3.13; no longer R42.1, R45.1, R46.2
- net N$11: now also IC3.12; no longer R47.1, R48.1, R52.2
- net N$12: now also IC3.11; no longer R49.1, R52.1, R53.2
- net N$13: now also IC7.17; no longer R50.1, R53.1, R54.2
- net N$2: now also C29.1
- net N$3: now also IC3.18, R31.1; no longer R33.1, R36.1, R37.2
- net N$4: now also C8.+, IC8.3; no longer X1.8
- net N$5: now also C9.+, IC8.5; no longer X1.7
- net N$6: now also C10.+, IC8.8; no longer X1.6
- net N$7: now also IC3.16, R33.1; no longer R34.1, R37.1, R38.2
- net N$8: now also IC3.15, R34.1; no longer R39.1, R40.1, R44.2
- net N$9: now also IC3.14; no longer R41.1, R44.1, R45.2
- net P1B1: now also K1.22; no longer JAMMA1.22, R15.2
- net P1B2: now also K1.23; no longer JAMMA1.23, R17.2
- net P1B3: now also K1.24; no longer JAMMA1.24, R19.2
- net P1B4: now also K1.25; no longer JAMMA1.25, R21.2
- net P1B5: now also K1.26; no longer JAMMA1.26, R13.2
- net P1DW: now also K1.19; no longer JAMMA1.19, R7.2
- net P1LH: now also K1.20; no longer JAMMA1.20, R9.2
- net P1RH: now also K1.21; no longer JAMMA1.21, R11.2
- net P1START: now also K1.17; no longer JAMMA1.17, R3.2
- net P1UP: now also K1.18; no longer JAMMA1.18, R5.2
- net R_AUDIO: now also X2.3; no longer R28.1
Routing:
- removed copper zone on layer 1, net GND
- removed copper zone on layer 16, net GND
Other:
- board size 120 x 145 mm -> 100 x 80 mm
- board text removed: "40 (10) 39 (11) 38 (NC) 37 (7) 36 (NC) 35 (NC) 34 (143) 33 (144) 32 (141) 31 (142) 30 (137) 29 (NC) 28 (135) 27 (136) 26 (132) 25 (133) 24 (GND) 23 (GND) 22 (129) 21 (128) 20 (127) 19 (126) 18 (125) 17 (NC) 16 (121) 15 (120) 14 (119) 13 (115) 12 (114) 11 (113) 10 (112) 09 (111) 08 (110) 07 (106) 06 (105) 05 (104) 04 (103) 03 (101) 02 (I/0) 01 (Vcc)"
- board text removed: "40 (30) 39 (28) 38 (32) 37 (31) 36 (NC) 35 (33) 34 (39) 33 (NC) 32 (43) 31 (42) 30 (46) 29 (44) 28 (50) 27 (49) 26 (52) 25 (51) 24 (GND) 23 (GND) 22 (54) 21 (53) 20 (58) 19 (55) 18 (60) 17 (59) 16 (65) 15 (64) 14 (67) 13 (66) 12 (69) 11 (68) 10 (71) 09 (NC) 08 (88) 07 (72) 06 (90) 05 (89) 04 (99) 03 (91) 02 (VCC) 01 (100)"
