File: board/eagle/MystiqueJamma.sch (EAGLE design)
At the start: 74 parts, among them IC1 7805, IC2 74LS245N, IC4 74LS245N, IC5 CY7C1049CV33, IC6 TDA1543T

Commit message: Shift registers to read controllers, new libs
Parts:
- removed B1: (no value), FPGA-BOARD:C4E6-K""
- removed JAMMA1: JAMMA_TOP, JAMMA:JAMMA_TOP
- removed JAMMA2: JAMMA_BOTTOM, JAMMA:JAMMA_BOTTOM
- removed X1: (no value), adafruit:F15HDH
- added C10, C8, C9: 10uF, rcl-2:CPOL-USE2.5-5
- added C11, C12, C13, C14, C15, C16, C17, C18, C19, C20, C21, C27, C28, C29, C7: 100nF, adafruit:C-USC1206
- added C22, C25, C26: (no value), rcl:CPOL-USE2-4
- added C23: 100u/25V, rcl:CPOL-USE3.5-8
- added C24: 1000u/25V, rcl:CPOL-USE3.5-8
- added D2, D3: (no value), diode:DIODE-SOD80C
- added IC10: TDA2030V, linear:TDA2030V
- added IC11: LA4425V, LA4425:LA4425V
- added IC3, IC7: 74LS245DW, 74xx-us:74LS245DW
- added IC8: (no value), TLS1233:TLS1233
- added IC9: 74HC4021D, 40xx:4021D
- added K1: JAMMA-EDGE, JAMMA:JAMMA-EDGE
- added R58: (no value), pot:TRIM_EU-B90P
- added R59, R60, R61, R62, R63, R64, R65, R66, R67, R68, R69, R70, R71, R72, R73, R74, R75, R76, R77, R78, R79, R80, R81, R82, R83, R84, R85, R86, R87, R88, R89, R90, R91, R92, R93: 330, adafruit:R-US_M1206
- added U$3: (no value), FPGA-BOARD:C4E6-K""
- added X2: 1503_09, con-lumberg:1503_09
- added X4: (no value), con-subd:HF15H
- C1: value 10uF -> 100uF
- C3: device adafruit:C-US025-025X050 -> adafruit:C-USC1206
- C5: device adafruit:C-US025-024X044 -> adafruit:C-USC1206
- IC2, IC4: value 74LS245N -> 74HC4021D; device 74xx-us:74LS245N -> 40xx:4021D
- R1, R3, R5: value 330 -> 470; device adafruit:R-US_0207/7 -> adafruit:R-US_R1206
- R10, R12, R14, R16, R18, R20, R22, R8: value 10k -> 330; device adafruit:R-US_0207/7 -> adafruit:R-US_M1206
- R11, R13, R15, R17, R19, R21, R29, R7: device adafruit:R-US_0207/7 -> adafruit:R-US_M1206
- R2, R4, R6: value 10k -> 470; device adafruit:R-US_0207/7 -> adafruit:R-US_R1206
- R23, R24, R25, R26, R27, R28: device adafruit:R-US_0207/7 -> adafruit:R-US_R1206
- R30: value 20k -> 330; device adafruit:R-US_0207/7 -> adafruit:R-US_M1206
- R31, R32, R33, R34, R35, R39, R40, R41, R42, R43, R47, R48, R49, R50, R51: value 2k -> 330; device adafruit:R-US_0207/7 -> adafruit:R-US_M1206
- R36, R37, R38, R44, R45, R46, R52, R53, R54: value 1k -> 330; device adafruit:R-US_0207/7 -> adafruit:R-US_M1206
- R55, R56: value 220 -> 330; device adafruit:R-US_0207/7 -> adafruit:R-US_M1206
- R57: value 220 -> (none); device adafruit:R-US_0207/7 -> pot:TRIM_EU-B90P
- R9: value 330 -> (none); device adafruit:R-US_0207/7 -> pot:3RP/1610N
Connections:
- net DAC_DATA renamed I2S_DATA
- net DAC_FSYNC renamed IS2_WS
- net DAC_SCK renamed I2S_BCK
- removed net +12: D1.A, JAMMA1.+12V
- removed net +5REG: C2.+, C3.1, IC1.OUT, IC6P1.VCC
- removed net 12+: JAMMA2.+12V
- removed net CS1_: IC2A.B1, R1.1, R2.1
- removed net CS1_3V: IC2A.A1
- removed net JVIDEO_BLUE: JAMMA1.VIDEO_BLUE, R55.2
- removed net JVIDEO_GREEN: JAMMA2.VIDEO_GREEN, R56.2
- removed net JVIDEO_RED: JAMMA1.VIDEO_RED, R57.2
- removed net P1B1_: IC2A.B7, R15.1, R16.1
- removed net P1B1_3V: IC2A.A7
- removed net P1B2_: IC2A.B8, R17.1, R18.1
- removed net P1B2_3V: IC2A.A8
- removed net P1B3_: IC4A.B1, R19.1, R20.1
- removed net P1B3_3V: IC4A.A1
- removed net P1B4_: IC4A.B2, R21.1, R22.1
- removed net P1B4_3V: IC4A.A2
- removed net P1B5_: IC4A.B3, R13.1, R14.1
- removed net P1B5_3V: IC4A.A3
- removed net P1D_: IC2A.B4, R7.1, R8.1
- removed net P1D_3V: IC2A.A4
- removed net P1L_: IC2A.B5, R10.1, R9.1
- removed net P1L_3V: IC2A.A5
- removed net P1R_: IC2A.B6, R11.1, R12.1
- removed net P1R_3V: IC2A.A6
- removed net P1S_: IC2A.B2, R3.1, R4.1
- removed net P1S_3V: IC2A.A2
- removed net P1U_: IC2A.B3, R5.1, R6.1
- removed net P1U_3V: IC2A.A3
- removed net SD_CS_144: B1B.7, U$2.CS
- removed net SD_DATAIN_142: B1B.9, R24.1, U$2.DATA_IN
- removed net SD_DATAOUT_141: B1B.10, R23.1, U$2.DATA_OUT
- removed net SD_SCLK_143: B1B.8, U$2.SCLK
- removed net VGA_B0: R47.2
- removed net VGA_B1: R49.2
- removed net VGA_B2: R50.2
- removed net VGA_B3: R51.2
- removed net VGA_BLUE: R51.1, R54.1, R55.1, X1.3
- removed net VGA_G0: R39.2
- removed net VGA_G1: R41.2
- removed net VGA_G2: R42.2
- removed net VGA_G3: R43.2
- removed net VGA_GREEN: R43.1, R46.1, R56.1, X1.2
- removed net VGA_HSYNC: JAMMA2.VIDEO_SYNC, X1.13
- removed net VGA_R0: R31.2
- removed net VGA_R1: R33.2
- removed net VGA_R2: R34.2
- removed net VGA_R3: R35.2
- removed net VGA_RED: R35.1, R38.1, R57.1, X1.1
- removed net VGA_VSYNC: X1.14
- new net +12V: C23.+, C27.1, D1.A, D3.C, IC10.V+, IC11.V+, IC8.VCC1, IC8.VCC2, K1PARTS.+12V, K1SOLDER.+12V, R2.1, R53.2, R54.2, R55.2
- new net +5V: C17.1, C18.1, C2.+, C3.1, C7.1, IC1.OUT, IC3P.VCC, IC6P1.VCC, IC7P.VCC
- new net B0: IC7A.A1
- new net B1: IC7A.A2
- new net B2: IC7A.A3
- new net B3: IC7A.A4
- new net BURST_GATE: IC8.!CLAMP_GATE
- new net CNTR_CLK: IC2A.CLK, IC4A.CLK, IC9A.CLK
- new net CNTR_DAT: IC2A.Q8
- new net CNTR_LATCH: IC2A.P/!S, IC4A.P/!S, IC9A.P/!S
- new net CSY: IC7A.A7
- new net G0: IC3A.A5
- new net G1: IC3A.A6
- new net G2: IC3A.A7
- new net G3: IC3A.A8
- new net GATE: IC7A.A8
- new net HSY: IC7A.A5
- new net JAMMA-BLUE: K1PARTS.VIDEO_BLUE, R52.2
- new net JAMMA-CSYNC: K1SOLDER.VIDEO_SYNC
- new net JAMMA-GREEN: K1SOLDER.VIDEO_GREEN, R51.2
- new net JAMMA-RED: K1PARTS.VIDEO_RED, R50.2
- new net JAMMA_AUDIO: R28.2, R29.2, R9.E
- new net LAA: R29.1, X2.4
- new net N$14: IC7A.B1
- new net N$15: IC7A.B3
- new net N$16: IC7A.B4
- new net N$17: IC7A.B5
- new net N$18: IC7A.B6
- new net N$19: IC7A.B7
- new net N$20: IC7A.B8
- new net N$21: C16.1, IC8.B-CLAMP, IC8.G-CLAMP, IC8.R-CLAMP, R58.S
- new net N$22: C11.1, IC8.R-CL_CAP
- new net N$23: C12.1, IC8.G-CL_CAP
- new net N$24: C13.1, IC8.B-CL_CAP
- new net N$25: IC8.R-OUT, R50.1, R59.2
- new net N$26: IC8.G-OUT, R51.1, R60.2, R61.2
- new net N$27: IC8.B-OUT, R52.1
- new net N$28: C14.1, IC8.CONTRAST, R57.S
- new net N$29: R53.1, R57.E
- new net N$30: IC2A.P1, R63.1
- new net N$31: R55.1, R58.E
- new net N$32: IC2A.P2, R7.1
- new net N$33: IC2A.P3, R8.1
- new net N$34: C15.1, IC8.B-GAIN, IC8.G-GAIN, IC8.R-GAIN, R54.1, R56.2
- new net N$35: IC2A.P4, R10.1
- new net N$36: IC2A.P5, R11.1
- new net N$37: IC2A.P6, R12.1
- new net N$38: IC2A.P7, R13.1
- new net N$39: IC2A.P8, R14.1
- new net N$40: IC4A.P1
- new net N$41: IC4A.P2
- new net N$42: IC4A.P3
- new net N$43: IC4A.P4
- new net N$44: IC4A.P5
- new net N$45: C22.+, R1.1, R2.2, R3.1
- new net N$46: R7.2
- new net N$47: R63.2
- new net N$48: IC4A.P6
- new net N$49: IC4A.P7
- new net N$50: IC4A.P8
- new net N$51: IC9A.P1
- new net N$52: IC9A.P2
- new net N$53: IC9A.P3
- new net N$54: IC9A.P4
- new net N$55: IC9A.P5
- new net N$56: IC9A.P6
- new net N$57: IC9A.P7
- new net N$58: IC9A.P8
- new net N$59: C28.1, R6.2
- new net N$60: C26.+, R4.2
- new net N$61: R8.2
- new net N$62: R10.2
- new net N$63: R12.2
- new net N$64: R11.2
- new net N$65: R13.2
- new net N$66: R14.2
- new net N$71: IC10.-IN, R4.1, R5.2
- new net N$88: IC2A.SI, IC4A.Q8
- new net N$89: IC4A.SI, IC9A.Q8
- new net N$91: C25.-, R9.S
- new net N$92: C25.+, IC10.+IN, IC11.+IN, R3.2
- new net N$93: C24.+, D2.C, D3.A, IC10.OUT, IC11.OUT, R5.1, R6.1
- new net R0: IC3A.A1
- new net R1: IC3A.A2
- new net R2: IC3A.A3
- new net R3: IC3A.A4
- new net RAA: R28.1, X2.5
- new net SD_CS: U$2.CS
- new net SD_DATAIN: R24.1, U$2.DATA_IN
- new net SD_DATAOUT: R23.1, U$2.DATA_OUT
- new net SD_SCLK: U$2.SCLK
- new net VGA-BLUE: C10.-, R35.2, X4.3
- new net VGA-GREEN: C9.-, R36.2, X4.2
- new net VGA-HSYNC: X4.13
- new net VGA-RED: C8.-, R31.2, R32.2, R33.2, R34.2, R47.2, X4.1
- new net VGA-VSYNC: X4.14
- new net VGA_DETECT: X4.5
- new net VSY: IC7A.A6
- net +3V3: now also C19.1, C20.1, C21.1, IC2P.VDD, IC4P.VDD, IC9P.VDD, R70.2, R71.2, R72.2, R73.2, R74.2, R75.2, R76.2, R77.2, R78.2, R79.2, R80.2, R81.2, R82.2, R83.2, R84.2, R85.2, R86.2, R87.2, R88.2, R89.2, R90.2, R91.2, R92.2, R93.2, U$3A.40, U$3B.39, U$3B.40; no longer B1A.40, B1B.39, B1B.40, IC2P.VCC, IC4P.VCC, R10.2, R12.2, R14.2, R16.2, R18.2, R2.2, R20.2, R22.2, R4.2, R6.2, R8.2
- net COINSW1: now also K1PARTS.COIN_SW1; no longer JAMMA1.COIN_SW1, R1.2
- net GND: now also C11.2, C12.2, C13.2, C14.2, C15.2, C16.2, C17.2, C18.2, C19.2, C20.2, C21.2, C22.-, C23.-, C26.-, C27.2, C28.2, C29.2, C7.2, D2.A, IC10.GND, IC11.-IN, IC11.GND, IC2P.VSS, IC3A.G, IC3P.GND, IC4P.VSS, IC7A.G, IC7P.GND, IC8.GND, IC9A.SI, IC9P.VSS, K1PARTS.GND@1, K1PARTS.GND@2, K1PARTS.GND@3, K1PARTS.GND@4, K1PARTS.VIDEO_GND, K1SOLDER.GND@1, K1SOLDER.GND@2, K1SOLDER.GND@3, K1SOLDER.GND@4, K1SOLDER.SPK-, R1.2, R35.1, R36.1, R47.1, R56.1, R57.A, R58.A, R59.1, R60.1, R61.1, R9.A, U$3A.17, U$3A.18, U$3B.17, U$3B.18, X2.1, X4.10, X4.6, X4.7, X4.8; no longer B1A.17, B1A.18, B1B.17, B1B.18, IC2A.DIR, IC2A.G, IC2P.GND, IC4A.DIR, IC4A.G, IC4P.GND, JAMMA1.GND@1, JAMMA1.GND@2, JAMMA1.GND@3, JAMMA1.GND@4, JAMMA1.VIDEO_GND, JAMMA2.GND@1, JAMMA2.GND@2, JAMMA2.GND@3, JAMMA2.GND@4, JAMMA2.SPK-, R30.1, R32.2, R40.2, R48.2, X1.10, X1.5
- net JAMMA_SPK+: now also C24.-, K1PARTS.SPK+; no longer JAMMA1.SPK+, R28.2, R29.2, R30.2
- net L_AUDIO: now also X2.2; no longer R29.1
- net N$1: now also IC3A.B2; no longer R31.1, R36.2
- net N$10: now also IC3A.B6; no longer R42.1, R45.1, R46.2
- net N$11: now also IC3A.B7; no longer R47.1, R48.1, R52.2
- net N$12: now also IC3A.B8; no longer R49.1, R52.1, R53.2
- net N$13: now also IC7A.B2; no longer R50.1, R53.1, R54.2
- net N$2: now also C29.1
- net N$3: now also IC3A.B1, R31.1; no longer R33.1, R36.1, R37.2
- net N$4: now also C8.+, IC8.R-IN; no longer X1.8
- net N$5: now also C9.+, IC8.G-IN; no longer X1.7
- net N$6: now also C10.+, IC8.B-IN; no longer X1.6
- net N$7: now also IC3A.B3, R33.1; no longer R34.1, R37.1, R38.2
- net N$8: now also IC3A.B4, R34.1; no longer R39.1, R40.1, R44.2
- net N$9: now also IC3A.B5; no longer R41.1, R44.1, R45.2
- net P1B1: now also K1PARTS.1P5_PUSH1; no longer JAMMA1.1P5_PUSH1, R15.2
- net P1B2: now also K1PARTS.1P6_PUSH2; no longer JAMMA1.1P6_PUSH2, R17.2
- net P1B3: now also K1PARTS.1P7_PUSH3; no longer JAMMA1.1P7_PUSH3, R19.2
- net P1B4: now also K1PARTS.1P8; no longer JAMMA1.1P8, R21.2
- net P1B5: now also K1PARTS.1P9; no longer JAMMA1.1P9, R13.2
- net P1DW: now also K1PARTS.1P2_DOWN; no longer JAMMA1.1P2_DOWN, R7.2
- net P1LH: now also K1PARTS.1P3_LEFT; no longer JAMMA1.1P3_LEFT, R9.2
- net P1RH: now also K1PARTS.1P4_RIGHT; no longer JAMMA1.1P4_RIGHT, R11.2
- net P1START: now also K1PARTS.START_SW1; no longer JAMMA1.START_SW1, R3.2
- net P1UP: now also K1PARTS.1P1_UP; no longer JAMMA1.1P1_UP, R5.2
- net R_AUDIO: now also X2.3; no longer R28.1
Other:
- note added: "AUDIO I2S BUS"
- note added: "CONTROLLER BUS"
- note added: "Mystique JAMMA"
- note added: "SRAM BUS"
- note added: "VIDEO BUS"
- moved on the sheet: C1, C2, C3, C4, C5, C6, D1, IC1, IC2P, IC4P, IC5, IC6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
