File: board/kicad/MystiqueJamma.kicad_pcb (KiCad board)
At the start: 2 copper layers, 154.2 x 144.8 mm, 110 parts, among them IC1 7805, IC10 74245N, IC2 74245N, IC3 74245N, IC4 74245N, IC5 CY7C1049CV33, IC6 TDA1543T, IC7 74245N, IC8 TLS1233, IC9 74245N, X2 1503_09, X4 HF15H

Commit message: kicad board layout
Parts:
- added REF**: MountingHole_4mm, MountingHole:MountingHole_4mm, F.Cu at (137.6, 212.6)
- added REF**: MountingHole_4mm, MountingHole:MountingHole_4mm, F.Cu at (271.1, 212.6)
- added REF**: MountingHole_4mm, MountingHole:MountingHole_4mm, F.Cu at (271.1, 76.8)
- added REF**: MountingHole_4mm, MountingHole:MountingHole_4mm, F.Cu at (137.6, 76.8)
- moved C2 224.6 mm to (156.6, 79.8), turned to 270 degrees
- moved C1 218.3 mm to (156.6, 86.4), turned to 90 degrees
- moved C5 214.0 mm to (162.6, 85.1), turned to 90 degrees
- moved C3 204.3 mm to (162.6, 78.7), turned to 270 degrees
- moved D1 98.0 mm to (142.2, 90.9)
- moved X4 96.5 mm to (264.2, 181.6)
- moved IC10 96.5 mm to (180.3, 191.8)
- moved IC2 96.5 mm to (208.3, 191.8)
- moved JAMMA1 96.5 mm to (127.0, 144.8)
- moved JAMMA2 96.5 mm to (127.0, 144.8)
- moved RN1 96.5 mm to (209.6, 184.2)
- moved RN2 96.5 mm to (181.6, 168.9)
- moved RN3 96.5 mm to (209.6, 168.9)
- moved RN4 96.5 mm to (181.6, 184.2)
- moved U$3 96.5 mm to (237.5, 121.9)
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Other:
- outline, holes or cut-outs redrawn

Commit message: kicad
Parts:
- moved C6 294.4 mm to (252.7, 137.2)
- moved C4 268.4 mm to (243.8, 137.2)
- moved C5 71.1 mm to (163.8, 14.0)
- moved C3 69.7 mm to (149.9, 10.2)
- moved D1 14.2 mm to (149.9, 102.9)

Commit message: FPGA board pins now defined
Parts:
- removed JAMMA1: JAMMA_TOP, MystiqueJamma:JAMMA_TOP
- removed JAMMA2: JAMMA_BOTTOM, MystiqueJamma:JAMMA_BOTTOM
- removed the REF** at (137.6, 212.6)
- removed the REF** at (271.1, 212.6)
- removed the REF** at (271.1, 76.8)
- removed the REF** at (137.6, 76.8)
- removed RN1, RN2, RN3, RN4: G08R, MystiqueJamma:SIL9
- added C23: 100u/25V, MystiqueJamma:E3,5-8, F.Cu at (62.9, 51.4)
- added C24: 1000u/25V, MystiqueJamma:E3,5-8, F.Cu at (54.0, 51.4)
- added C25: CPOL-USE2-4, MystiqueJamma:E2-4, F.Cu at (125.7, 92.7)
- added C26: CPOL-USE2-4, MystiqueJamma:E2-4, F.Cu at (60.3, 61.6)
- added C27: 100nF, MystiqueJamma:C1206, B.Cu at (47.0, 49.5)
- added C28: 100nF, MystiqueJamma:C1206, B.Cu at (47.6, 60.3)
- added C29: 100nF, MystiqueJamma:C1206, B.Cu at (81.9, 42.5)
- added D2: DIODE-SOD80C, MystiqueJamma:SOD80C, F.Cu at (56.5, 57.8)
- added D3: DIODE-SOD80C, MystiqueJamma:SOD80C, F.Cu at (62.9, 57.8)
- added IC11: LA4425V, MystiqueJamma:LA4425, F.Cu at (58.4, 38.1)
- added K1: JAMMA-EDGE, MystiqueJamma:JAMMA-EDGE, F.Cu at (22.2, 38.7)
- added R10: 330, MystiqueJamma:M1206, F.Cu at (50.8, 79.5)
- added R11: 330, MystiqueJamma:M1206, F.Cu at (50.8, 73.4)
- added R12: 330, MystiqueJamma:M1206, F.Cu at (50.8, 70.4)
- added R13: 330, MystiqueJamma:M1206, F.Cu at (50.8, 67.3)
- added R14: 330, MystiqueJamma:M1206, F.Cu at (50.8, 76.5)
- added R15: 330, MystiqueJamma:M1206, F.Cu at (50.8, 113.0)
- added R16: 330, MystiqueJamma:M1206, F.Cu at (50.8, 110.0)
- added R17: 330, MystiqueJamma:M1206, F.Cu at (50.8, 106.9)
- added R18: 330, MystiqueJamma:M1206, F.Cu at (50.8, 103.9)
- added R19: 330, MystiqueJamma:M1206, F.Cu at (50.8, 97.8)
- added R2: 470, MystiqueJamma:R1206, B.Cu at (44.5, 41.3)
- added R20: 330, MystiqueJamma:M1206, F.Cu at (50.8, 94.7)
- added R21: 330, MystiqueJamma:M1206, F.Cu at (50.8, 91.7)
- added R22: 330, MystiqueJamma:M1206, F.Cu at (50.8, 100.8)
- added R3: 470, MystiqueJamma:R1206, B.Cu at (50.2, 45.1)
- added R4: 470, MystiqueJamma:R1206, B.Cu at (54.0, 61.0)
- added R5: 470, MystiqueJamma:R1206, B.Cu at (47.0, 57.1)
- added R6: 470, MystiqueJamma:R1206, B.Cu at (47.0, 53.3)
- added R7: 330, MystiqueJamma:M1206, F.Cu at (50.8, 85.6)
- added R8: 330, MystiqueJamma:M1206, F.Cu at (50.9, 82.5)
- added R89: 330, MystiqueJamma:M1206, F.Cu at (56.1, 128.3)
- added R9: 3RP_1610N, MystiqueJamma:3RP_1610N, F.Cu at (134.6, 92.7)
- added R90: 330, MystiqueJamma:M1206, F.Cu at (56.1, 122.2)
- added R91: 330, MystiqueJamma:M1206, F.Cu at (56.1, 119.1)
- added R92: 330, MystiqueJamma:M1206, F.Cu at (56.1, 116.1)
- added R93: 330, MystiqueJamma:M1206, F.Cu at (56.1, 125.2)
- added REF**: MountingHole_4mm, Mounting_Holes:MountingHole_4mm, F.Cu at (111.0, 145.3)
- added REF**: MountingHole_4mm, Mounting_Holes:MountingHole_4mm, F.Cu at (100.8, 40.4)
- C1: value 10uF -> 100uF; footprint MystiqueJamma:E2,5-5 -> MystiqueJamma:E2,5-7
- C11, C12, C13, C19, C20, C21, C5: footprint MystiqueJamma:C025-024X044 -> MystiqueJamma:C1206
- C14, C15, C16, C17, C18, C7: footprint MystiqueJamma:C025-024X044 -> MystiqueJamma:C1206; moved to B.Cu
- C22: value 100nF -> CPOL-USE2-4; footprint MystiqueJamma:C025-024X044 -> MystiqueJamma:E2-4
- C3: footprint MystiqueJamma:C025-025X050 -> MystiqueJamma:C1206
- C4, C6: footprint MystiqueJamma:E5-6 -> MystiqueJamma:E2-4
- IC10: value 74245N -> TDA2030V; footprint MystiqueJamma:DIL20 -> MystiqueJamma:CB360
- IC2, IC4, IC9: value 74245N -> 74HC4021D; footprint MystiqueJamma:DIL20 -> MystiqueJamma:SO16
- IC3, IC7: value 74245N -> 74LS245DW; footprint MystiqueJamma:DIL20 -> MystiqueJamma:SO20W
- R1: value 330 -> 470; footprint MystiqueJamma:0207_7 -> MystiqueJamma:R1206; moved to B.Cu
- R23, R24, R25, R26, R27, R28: footprint MystiqueJamma:0207_7 -> MystiqueJamma:R1206
- R29, R62, R63, R64, R65, R66, R67, R68, R69, R70, R71, R72, R73, R74, R75, R76, R77, R78, R79, R80, R81, R82, R83, R84, R85, R86, R87, R88: footprint MystiqueJamma:0207_7 -> MystiqueJamma:M1206
- R30: value 20k -> 330; footprint MystiqueJamma:0207_7 -> MystiqueJamma:M1206
- R31, R36: value 330 -> 420; footprint MystiqueJamma:0207_7 -> MystiqueJamma:M1206; moved to B.Cu
- R32, R37: value 330 -> 785; footprint MystiqueJamma:0207_7 -> MystiqueJamma:M1206; moved to B.Cu
- R33, R38: value 330 -> 1380; footprint MystiqueJamma:0207_7 -> MystiqueJamma:M1206; moved to B.Cu
- R34, R39: value 330 -> 2230; footprint MystiqueJamma:0207_7 -> MystiqueJamma:M1206; moved to B.Cu
- R35, R41, R42, R43, R44, R45, R46, R48, R49, R50, R51, R52, R53, R54, R55, R56, R59, R60, R61: footprint MystiqueJamma:0207_7 -> MystiqueJamma:M1206; moved to B.Cu
- R40, R47: value 330 -> 125; footprint MystiqueJamma:0207_7 -> MystiqueJamma:M1206; moved to B.Cu
- moved R47 292.5 mm to (120.7, 61.0), turned to 270 degrees
- moved R49 275.1 mm to (108.0, 78.1), turned to 90 degrees
- moved R48 269.2 mm to (111.1, 78.1), turned to 270 degrees
- moved R46 263.6 mm to (114.3, 78.1), turned to 270 degrees
- moved R45 262.0 mm to (117.5, 78.1), turned to 270 degrees
- moved R44 256.1 mm to (108.0, 72.4), turned to 270 degrees
- moved R43 254.5 mm to (111.1, 72.3), turned to 270 degrees
- moved R40 254.3 mm to (120.7, 66.7), turned to 270 degrees
- moved R42 252.9 mm to (114.3, 72.4), turned to 270 degrees
- moved R41 251.6 mm to (117.5, 72.4), turned to 270 degrees
- moved C14 250.7 mm to (114.3, 47.6), turned to 90 degrees
- moved C16 247.3 mm to (117.5, 47.6), turned to 90 degrees
- moved C15 244.8 mm to (111.1, 47.6), turned to 90 degrees
- moved R39 241.7 mm to (108.0, 66.7), turned to 270 degrees
- moved R38 240.4 mm to (111.1, 66.7), turned to 270 degrees
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Connections:
- IC10 pad 2: /BTN-5 -> Net-(IC10-Pad2)
- IC10 pad 3: /BTN-6 -> GND
- IC10 pad 4: /COIN_SW -> Net-(C24-Pad+)
- IC10 pad 5: /START -> +12V
- IC2 pad 10: GND -> /CNTR_CLK
- IC2 pad 16: Net-(IC2-Pad16) -> +3V3
- IC2 pad 2: /UP -> Net-(IC2-Pad2)
- IC2 pad 3: /DOWN -> /CNTR_DAT
- IC2 pad 4: /LEFT -> Net-(IC2-Pad4)
- IC2 pad 5: /RIGHT -> Net-(IC2-Pad5)
- IC2 pad 6: /BTN-1 -> Net-(IC2-Pad6)
- IC2 pad 7: /BTN-2 -> Net-(IC2-Pad7)
- IC2 pad 8: /BTN-3 -> GND
- IC2 pad 9: /BTN-4 -> /CNTR_LATCH
- IC4 pad 10: GND -> /CNTR_CLK
- IC4 pad 16: Net-(IC4-Pad16) -> +3V3
- IC4 pad 2: /BTN-5 -> Net-(IC4-Pad2)
- IC4 pad 3: /BTN-6 -> Net-(IC2-Pad11)
- IC4 pad 4: /COIN_SW -> Net-(IC4-Pad4)
- IC4 pad 5: /START -> Net-(IC4-Pad5)
- IC4 pad 6: /COIN_COUNT -> Net-(IC4-Pad6)
- IC4 pad 8: Net-(IC4-Pad8) -> GND
- IC4 pad 9: Net-(IC4-Pad9) -> /CNTR_LATCH
- IC9 pad 10: GND -> /CNTR_CLK
- IC9 pad 11: Net-(IC9-Pad11) -> GND
- IC9 pad 16: Net-(IC9-Pad16) -> +3V3
- IC9 pad 2: /UP -> Net-(IC9-Pad2)
- IC9 pad 3: /DOWN -> Net-(IC4-Pad11)
- IC9 pad 4: /LEFT -> Net-(IC9-Pad4)
- IC9 pad 5: /RIGHT -> Net-(IC9-Pad5)
- IC9 pad 6: /BTN-1 -> Net-(IC9-Pad6)
- IC9 pad 7: /BTN-2 -> Net-(IC9-Pad7)
- IC9 pad 8: /BTN-3 -> GND
- IC9 pad 9: /BTN-4 -> /CNTR_LATCH
- R1 pad 1: Net-(IC10-Pad12) -> Net-(C22-Pad+)
- R1 pad 2: /VGA_DETECT -> GND
- R30 pad 1: GND -> Net-(IC9-Pad7)
- R30 pad 2: /JAMMA_AUDIO -> /N$75
- R35 pad 1: Net-(IC3-Pad14) -> GND
- R35 pad 2: /VGA-GREEN -> /VGA-BLUE
- R36 pad 1: Net-(IC3-Pad13) -> Net-(IC3-Pad14)
- R37 pad 1: Net-(IC3-Pad12) -> Net-(IC3-Pad13)
- R38 pad 1: Net-(IC3-Pad11) -> Net-(IC3-Pad12)
- R39 pad 1: Net-(IC7-Pad17) -> Net-(IC3-Pad11)
- R39 pad 2: /VGA-BLUE -> /VGA-GREEN
- R40 pad 1: Net-(IC7-Pad18) -> GND
- R40 pad 2: /VGA-BLUE -> /VGA-GREEN
- R41 pad 1: Net-(IC7-Pad16) -> Net-(IC7-Pad18)
- R42 pad 1: Net-(IC7-Pad15) -> Net-(IC7-Pad17)
- R43 pad 1: Net-(IC7-Pad14) -> Net-(IC7-Pad16)
- R43 pad 2: /VGA-HSYNC -> /VGA-BLUE
- R44 pad 1: Net-(IC7-Pad13) -> Net-(IC7-Pad15)
- R44 pad 2: /VGA-VSYNC -> /VGA-BLUE
- R45 pad 1: Net-(IC7-Pad12) -> Net-(IC7-Pad14)
- R45 pad 2: /JAMMA-CSYNC -> /VGA-HSYNC
- R46 pad 1: Net-(IC7-Pad11) -> Net-(IC7-Pad13)
- R46 pad 2: /BURST_GATE -> /VGA-VSYNC
- R48 pad 1: GND -> Net-(IC7-Pad12)
- R48 pad 2: /VGA-GREEN -> /JAMMA-CSYNC
- R49 pad 1: GND -> Net-(IC7-Pad11)
- R49 pad 2: /VGA-BLUE -> /BURST_GATE
- R52 pad 2: /JAMA-BLUE -> /JAMMA-BLUE
- R61 pad 2: Net-(IC8-Pad15) -> Net-(IC8-Pad13)
- R62 pad 1: Net-(IC2-Pad17) -> Net-(IC9-Pad6)
- R62 pad 2: /N$46 -> /N$77
- R63 pad 1: Net-(IC2-Pad18) -> Net-(IC2-Pad7)
- R64 pad 1: Net-(IC2-Pad16) -> Net-(IC9-Pad5)
- R64 pad 2: /N$61 -> /N$78
- R65 pad 1: Net-(IC2-Pad15) -> Net-(IC9-Pad4)
- R65 pad 2: /N$62 -> /N$80
- R66 pad 1: Net-(IC2-Pad13) -> Net-(IC9-Pad13)
- R66 pad 2: /N$63 -> /N$79
- R67 pad 1: Net-(IC2-Pad14) -> Net-(IC9-Pad14)
- R67 pad 2: /N$64 -> /N$81
- R68 pad 1: Net-(IC2-Pad12) -> Net-(IC9-Pad15)
- R68 pad 2: /N$65 -> /N$82
- R69 pad 1: Net-(IC2-Pad11) -> Net-(IC9-Pad1)
- R69 pad 2: /N$66 -> /VGA_DETECT
- R70 pad 1: Net-(IC4-Pad17) -> Net-(IC2-Pad7)
- R70 pad 2: /N$67 -> +3V3
- R71 pad 1: Net-(IC4-Pad18) -> Net-(IC2-Pad6)
- R71 pad 2: /N$68 -> +3V3
- R72 pad 1: Net-(IC4-Pad16) -> Net-(IC2-Pad5)
- R72 pad 2: /N$69 -> +3V3
- R73 pad 1: Net-(IC4-Pad15) -> Net-(IC2-Pad4)
- R73 pad 2: /N$70 -> +3V3
- R74 pad 1: Net-(IC10-Pad13) -> Net-(IC2-Pad13)
- R74 pad 2: /N$71 -> +3V3
- R75 pad 1: Net-(IC4-Pad14) -> Net-(IC2-Pad14)
- R75 pad 2: /N$72 -> +3V3
- R76 pad 1: Net-(IC9-Pad18) -> Net-(IC2-Pad15)
- R76 pad 2: /N$73 -> +3V3
- R77 pad 1: Net-(IC9-Pad17) -> Net-(IC2-Pad1)
- R77 pad 2: /N$74 -> +3V3
- R78 pad 1: Net-(IC9-Pad15) -> Net-(IC4-Pad7)
- R78 pad 2: /N$75 -> +3V3
- R79 pad 1: Net-(IC9-Pad16) -> Net-(IC4-Pad6)
- R79 pad 2: /N$76 -> +3V3
- R80 pad 1: Net-(IC9-Pad14) -> Net-(IC4-Pad5)
- R80 pad 2: /N$77 -> +3V3
- R81 pad 1: Net-(IC9-Pad13) -> Net-(IC4-Pad4)
- R81 pad 2: /N$78 -> +3V3
- R82 pad 1: Net-(IC9-Pad11) -> Net-(IC4-Pad13)
- R82 pad 2: /N$79 -> +3V3
- R83 pad 1: Net-(IC9-Pad12) -> Net-(IC4-Pad14)
- R83 pad 2: /N$80 -> +3V3
- R84 pad 1: Net-(IC10-Pad18) -> Net-(IC4-Pad15)
- R84 pad 2: /N$81 -> +3V3
- R85 pad 1: Net-(IC10-Pad17) -> Net-(IC4-Pad1)
- R85 pad 2: /N$82 -> +3V3
- R86 pad 1: Net-(IC10-Pad15) -> Net-(IC9-Pad7)
- R86 pad 2: /N$83 -> +3V3
- R87 pad 1: Net-(IC10-Pad16) -> Net-(IC9-Pad6)
- R87 pad 2: /N$84 -> +3V3
- R88 pad 1: Net-(IC10-Pad14) -> Net-(IC9-Pad5)
- R88 pad 2: /N$85 -> +3V3
Routing:
- net /COINSW1: track 0.00 -> 50.9 mm
- net /P1START: track 0.00 -> 48.9 mm
- net /P1UP: track 0.00 -> 46.5 mm
- net /P1DW: track 0.00 -> 39.8 mm
- net /P1LH: track 0.00 -> 36.0 mm
- net /P1RH: track 0.00 -> 29.8 mm
- net /P1B1: track 0.00 -> 25.9 mm
- net /P1B2: track 0.00 -> 21.5 mm
- net /P1B3: track 0.00 -> 17.8 mm
- net /P1B4: track 0.00 -> 11.6 mm
- net /P1B5: track 0.00 -> 8.10 mm
Other:
- board size 154.2 x 144.8 mm -> 106.7 x 116.2 mm
- net class Default: trace_width 0.25 -> 0.254; via_dia 0.8 -> 0.5; via_drill 0.4 -> 0.3
- net class POWER added: clearance 0.2, trace_width 0.6096, via_dia 0.6096, via_drill 0.6
- net class POWER2 added: clearance 0.2, trace_width 0.4064, via_dia 0.5, via_drill 0.3
