File: board/kicad/MystiqueJamma.sch (KiCad schematic (older format))
At the start: 110 parts, among them IC1 7805, IC10 74245N, IC2 74245N, IC3 74245N, IC4 74245N, IC5 CY7C1049CV33, IC6 TDA1543T, IC7 74245N, IC8 TLS1233, IC9 74245N, X2 1503_09, X4 HF15H

Commit message: FPGA board pins now defined
Parts:
- removed C1: 10uF, MystiqueJamma:E2,5-5, symbol MystiqueJamma-eagle-import:CPOL-USE2.5-5
- removed C22: 100nF, MystiqueJamma:C025-024X044, symbol MystiqueJamma-eagle-import:C-US025-024X044
- removed unit 2 of IC10
- removed IC2, IC3, IC4, IC7, IC9: 74245N, MystiqueJamma:DIL20, symbol MystiqueJamma-eagle-import:74245N
- removed JAMMA1: JAMMA_TOP, MystiqueJamma:JAMMA_TOP, symbol MystiqueJamma-eagle-import:JAMMA_TOP
- removed JAMMA2: JAMMA_BOTTOM, MystiqueJamma:JAMMA_BOTTOM, symbol MystiqueJamma-eagle-import:JAMMA_BOTTOM
- removed R1, R31, R32, R33, R34, R36, R37, R38, R39, R40, R47: 330, MystiqueJamma:0207_7, symbol MystiqueJamma-eagle-import:R-US_0207_7
- removed R30: 20k, MystiqueJamma:0207_7, symbol MystiqueJamma-eagle-import:R-US_0207_7
- removed RN1, RN2, RN3, RN4: G08R, MystiqueJamma:SIL9, symbol MystiqueJamma-eagle-import:G08R
- added C1: 100uF, MystiqueJamma:E2,5-7, symbol MystiqueJamma-eagle-import:CPOL-USE2.5-7
- added C22, C25, C26: CPOL-USE2-4, MystiqueJamma:E2-4, symbol MystiqueJamma-eagle-import:CPOL-USE2-4
- added C23: 100u/25V, MystiqueJamma:E3,5-8, symbol MystiqueJamma-eagle-import:CPOL-USE3.5-8
- added C24: 1000u/25V, MystiqueJamma:E3,5-8, symbol MystiqueJamma-eagle-import:CPOL-USE3.5-8
- added C27, C28, C29: 100nF, MystiqueJamma:C1206, symbol MystiqueJamma-eagle-import:C-USC1206
- added D2, D3: DIODE-SOD80C, MystiqueJamma:SOD80C, symbol MystiqueJamma-eagle-import:DIODE-SOD80C
- added IC11: LA4425V, MystiqueJamma:LA4425, symbol MystiqueJamma-eagle-import:LA4425V
- added IC2, IC4, IC9: 74HC4021D, MystiqueJamma:SO16, symbol MystiqueJamma-eagle-import:4021D
- added IC3, IC7: 74LS245DW, MystiqueJamma:SO20W, symbol MystiqueJamma-eagle-import:74245DW
- added K1: JAMMA-EDGE, MystiqueJamma:JAMMA-EDGE, symbol MystiqueJamma-eagle-import:JAMMA-EDGE
- added R1, R2, R3, R4, R5, R6: 470, MystiqueJamma:R1206, symbol MystiqueJamma-eagle-import:R-US_R1206
- added R10, R11, R12, R13, R14, R15, R16, R17, R18, R19, R20, R21, R22, R30, R7, R8, R89, R90, R91, R92, R93: 330, MystiqueJamma:M1206, symbol MystiqueJamma-eagle-import:R-US_M1206
- added R31, R36: 420, MystiqueJamma:M1206, symbol MystiqueJamma-eagle-import:R-US_M1206
- added R32, R37: 785, MystiqueJamma:M1206, symbol MystiqueJamma-eagle-import:R-US_M1206
- added R33, R38: 1380, MystiqueJamma:M1206, symbol MystiqueJamma-eagle-import:R-US_M1206
- added R34, R39: 2230, MystiqueJamma:M1206, symbol MystiqueJamma-eagle-import:R-US_M1206
- added R40, R47: 125, MystiqueJamma:M1206, symbol MystiqueJamma-eagle-import:R-US_M1206
- added R9: 3RP_1610N, MystiqueJamma:3RP_1610N, symbol MystiqueJamma-eagle-import:3RP_1610N
- C11, C12, C13, C14, C15, C16, C17, C18, C19, C20, C21, C5, C7: footprint MystiqueJamma:C025-024X044 -> MystiqueJamma:C1206; symbol MystiqueJamma-eagle-import:C-US025-024X044 -> MystiqueJamma-eagle-import:C-USC1206
- C3: footprint MystiqueJamma:C025-025X050 -> MystiqueJamma:C1206; symbol MystiqueJamma-eagle-import:C-US025-025X050 -> MystiqueJamma-eagle-import:C-USC1206
- C4, C6: footprint MystiqueJamma:E5-6 -> MystiqueJamma:E2-4; symbol MystiqueJamma-eagle-import:CPOL-USE5-6 -> MystiqueJamma-eagle-import:CPOL-USE2-4
- IC10: value 74245N -> TDA2030V; footprint MystiqueJamma:DIL20 -> MystiqueJamma:CB360; symbol MystiqueJamma-eagle-import:74245N -> MystiqueJamma-eagle-import:TDA2030V
- R23, R24, R25, R26, R27, R28: footprint MystiqueJamma:0207_7 -> MystiqueJamma:R1206; symbol MystiqueJamma-eagle-import:R-US_0207_7 -> MystiqueJamma-eagle-import:R-US_R1206
- R29, R35, R41, R42, R43, R44, R45, R46, R48, R49, R50, R51, R52, R53, R54, R55, R56, R59, R60, R61, R62, R63, R64, R65, R66, R67, R68, R69, R70, R71, R72, R73, R74, R75, R76, R77, R78, R79, R80, R81, R82, R83, R84, R85, R86, R87, R88: footprint MystiqueJamma:0207_7 -> MystiqueJamma:M1206; symbol MystiqueJamma-eagle-import:R-US_0207_7 -> MystiqueJamma-eagle-import:R-US_M1206
- U$3: symbol MystiqueJamma-eagle-import:C4E6-K__ -> MystiqueJamma-rescue:C4E6-K__-MystiqueJamma-eagle-import
Connections:
- net labels added: CNTR_CLK, CNTR_DAT, CNTR_LATCH, JAMMA-BLUE
- net labels removed: 2P-SELECT, BTN-1, BTN-2, BTN-3, BTN-4, BTN-5, BTN-6, COIN_COUNT, COIN_SW, DOWN, JAMA-BLUE, JVIDEO_BLUE, JVIDEO_GREEN, JVIDEO_RED, LEFT, N$71, N$83, N$84, N$85, RIGHT, START, TILT_SW, UP, VGA_HSYNC, VIDEOMODE
- wire segments 513 -> 663
- no-connect marks 0 -> 11
