File: board/Kicad/MystiqueJamma.sch (KiCad schematic (older format))
At the start: 163 parts, among them IC1 7805, IC10 TDA2030V, IC11 LA4425V, IC12 CY7C1049CV33, IC2 74HC4021D, IC3 74LS245DW, IC4 74HC4021D, IC5 CY7C1049CV33, IC6 TDA1543T, IC7 74LS245DW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

Commit message: Circuit update and cleanup
Added second SRAM, changed VGA detect to FPGA instead of shift registers, added solder joint to force VGA mode, added RC-Network to Shift Register clock signal to allow same line to control LATCH signal.
Parts:
- added unit 3 of EVB1
Connections:
- net VGA_DET_IN: now reaches D4.A, D5.C, R94.1, R95.1
- net VGA_DET_IN: now also EVB1.I0_91 (37); no longer IC9.11 (SI)
- no-connect marks 47 -> 46
Other:
- moved on the sheet: D4, D5, R94, R95
Changed lines of the file:
@@
 Sheet 1 1
 Title "Mystique Jamma"
-Date "2018-11-23"
+Date "2018-12-04"
 Rev "A"
 Comp "Reinaldo Flamino / Danjovic"
@@
 JAMMA-CSYNC
 Wire Wire Line
-	9400 6400 10500 6400
+	9400 6400 10300 6400
 Wire Wire Line
 	5400 3200 5700 3200
@@
 Text Label 18100 12200 0    50   ~ 0
 COINSW1
-Text Label 10500 6400 0    70   ~ 0
+Text Label 9750 6400 0    70   ~ 0
 VGA_DETECT
 $Comp
 L MystiqueJamma-eagle-import:R-US_M1206 R95
 U 1 0 5C424341
-P 16950 13050
-F 0 "R95" H 16900 13150 59  0000 L BNN
-F 1 "330" H 17090 13060 59  0000 L BNN
-F 2 "MystiqueJamma:M1206" H 16950 13050 50  0001 C CNN
-F 3 "" H 16950 13050 50  0001 C CNN
-	1    16950 13050
+P 6150 7150
+F 0 "R95" H 6100 7250 59  0000 L BNN
+F 1 "330" H 6290 7160 59  0000 L BNN
+F 2 "MystiqueJamma:M1206" H 6150 7150 50  0001 C CNN
+F 3 "" H 6150 7150 50  0001 C CNN
+	1    6150 7150
 	1    0    0    -1
 $EndComp
-Wire Wire Line
-	17150 13050 17550 13050
 $Comp
 L MystiqueJamma-eagle-import:R-US_M1206 R94
 U 1 0 5C5E40AD
-P 16600 12750
-F 0 "R94" V 16700 12500 59  0000 L BNN
-F 1 "10k" V 16600 12500 59  0000 L BNN
-F 2 "MystiqueJamma:M1206" H 16600 12750 50  0001 C CNN
-F 3 "" H 16600 12750 50  0001 C CNN
-	1    16600 12750
+P 5800 6850
+F 0 "R94" V 5900 6600 59  0000 L BNN
+F 1 "10k" V 5800 6600 59  0000 L BNN
+F 2 "MystiqueJamma:M1206" H 5800 6850 50  0001 C CNN
+F 3 "" H 5800 6850 50  0001 C CNN
+	1    5800 6850
 	0    -1   -1   0
 $EndComp
@@
 L MystiqueJamma-eagle-import:DIODE-SOD80C D5
 U 1 0 5CA8F8CB
-P 16300 13250
-F 0 "D5" V 16350 13350 59  0000 L BNN
-F 1 "4148" V 16250 13350 59  0000 L BNN
-F 2 "MystiqueJamma:SOD80C" H 16300 13250 50  0001 C CNN
-F 3 "" H 16300 13250 50  0001 C CNN
-	1    16300 13250
+P 5500 7350
+F 0 "D5" V 5550 7450 59  0000 L BNN
+F 1 "4148" V 5450 7450 59  0000 L BNN
+F 2 "MystiqueJamma:SOD80C" H 5500 7350 50  0001 C CNN
+F 3 "" H 5500 7350 50  0001 C CNN
+	1    5500 7350
 	0    -1   -1   0
 $EndComp
@@
 L MystiqueJamma-eagle-import:+3V3 #+3V0101
 U 1 0 5CB25249
-P 16600 12350
-F 0 "#+3V0101" H 16600 12350 50  0001 C CNN
-F 1 "+3V3" V 16500 12150 59  0000 L BNN
-F 2 "" H 16600 12350 50  0001 C CNN
-F 3 "" H 16600 12350 50  0001 C CNN
-	1    16600 12350
+P 5800 6450
+F 0 "#+3V0101" H 5800 6450 50  0001 C CNN
+F 1 "+3V3" H 5850 6450 59  0000 L BNN
+F 2 "" H 5800 6450 50  0001 C CNN
+F 3 "" H 5800 6450 50  0001 C CNN
+	1    5800 6450
 	1    0    0    -1
 $EndComp
@@
 L MystiqueJamma-eagle-import:GND #GND0103
 U 1 0 5CB25384
-P 16300 13550
-F 0 "#GND0103" H 16300 13550 50  0001 C CNN
-F 1 "GND" H 16200 13450 59  0000 L BNN
-F 2 "" H 16300 13550 50  0001 C CNN
-F 3 "" H 16300 13550 50  0001 C CNN
-	1    16300 13550
+P 5500 7650
+F 0 "#GND0103" H 5500 7650 50  0001 C CNN
+F 1 "GND" H 5400 7550 59  0000 L BNN
+F 2 "" H 5500 7650 50  0001 C CNN
+F 3 "" H 5500 7650 50  0001 C CNN
+	1    5500 7650
 	1    0    0    -1
 $EndComp
 Wire Wire Line
-	16750 13050 16600 13050
+	5950 7150 5800 7150
 Wire Wire Line
-	16600 12950 16600 13050
+	5800 7050 5800 7150
 Wire Wire Line
-	16600 12450 16600 12500
+	5800 6550 5800 6600
 Wire Wire Line
-	16600 12500 16300 12500
+	5800 6600 5500 6600
 Wire Wire Line
-	16300 12500 16300 12650
-Connection ~ 16600 12500
+	5500 6600 5500 6750
+Connection ~ 5800 6600
 Wire Wire Line
-	16600 12500 16600 12550
+	5800 6600 5800 6650
 $Comp
 L MystiqueJamma-eagle-import:DIODE-SOD80C D4
 U 1 0 5CEB07EB
-P 16300 12750
-F 0 "D4" V 16350 12850 59  0000 L BNN
-F 1 "4148" V 16250 12850 59  0000 L BNN
-F 2 "MystiqueJamma:SOD80C" H 16300 12750 50  0001 C CNN
-F 3 "" H 16300 12750 50  0001 C CNN
-	1    16300 12750
+P 5500 6850
+F 0 "D4" V 5550 6950 59  0000 L BNN
+F 1 "4148" V 5450 6950 59  0000 L BNN
+F 2 "MystiqueJamma:SOD80C" H 5500 6850 50  0001 C CNN
+F 3 "" H 5500 6850 50  0001 C CNN
+	1    5500 6850
 	0    -1   -1   0
 $EndComp
-Text Label 17550 13050 0    70   ~ 0
+Text Label 6750 7150 0    70   ~ 0
 VGA_DETECT
-Connection ~ 16600 13050
+Connection ~ 5800 7150
 Wire Wire Line
 	15900 12400 15900 13050
@@
 	15500 12400 15900 12400
 Wire Wire Line
-	15900 13050 16300 13050
-Wire Wire Line
-	16600 13050 16300 13050
-Connection ~ 16300 13050
+	5800 7150 5500 7150
+Connection ~ 5500 7150
 Wire Wire Line
-	16300 13050 16300 13150
+	5500 7150 5500 7250
 Wire Wire Line
-	16300 12850 16300 13050
+	5500 6950 5500 7150
 Wire Wire Line
-	16300 13350 16300 13450
+	5500 7450 5500 7550
 Text Label 19400 11200 2    70   ~ 0
 GND
@@
 L MystiqueJamma-rescue:Conn_01x02_Male-Connector J3
 U 1 1 5BED1A57
-P 2300 3450
-F 0 "J3" H 2406 3628 50  0000 C CNN
-F 1 "FPGA PWR" H 2406 3537 50  0000 C CNN
-F 2 "Connector_PinHeader_2.54mm:PinHeader_1x02_P2.54mm_Horizontal" H 2300 3450 50  0001 C CNN
-F 3 "~" H 2300 3450 50  0001 C CNN
-	1    2300 3450
-	1    0    0    -1
+P 2300 3550
+F 0 "J3" H 2400 3250 50  0000 C CNN
+F 1 "FPGA PWR" H 2400 3350 50  0000 C CNN
+F 2 "Connector_PinHeader_2.54mm:PinHeader_1x02_P2.54mm_Horizontal" H 2300 3550 50  0001 C CNN
+F 3 "~" H 2300 3550 50  0001 C CNN
+	1    2300 3550
+	1    0    0    1
 $EndComp
 $Comp
@@
 PS2DAT
 NoConn ~ 3000 10400
-NoConn ~ 3000 10500
 NoConn ~ 3900 10400
 Text Label 2400 10100 0    50   ~ 0
@@
 L MystiqueJamma-eagle-import:GND #GND032
 U 1 0 5C75BDBC
-P 14700 13400
-F 0 "#GND032" H 14700 13400 50  0001 C CNN
-F 1 "GND" H 14600 13300 59  0000 L BNN
-F 2 "" H 14700 13400 50  0001 C CNN
-F 3 "" H 14700 13400 50  0001 C CNN
-	1    14700 13400
+P 15900 13150
+F 0 "#GND032" H 15900 13150 50  0001 C CNN
+F 1 "GND" H 15800 13050 59  0000 L BNN
+F 2 "" H 15900 13150 50  0001 C CNN
+F 3 "" H 15900 13150 50  0001 C CNN
+	1    15900 13150
 	1    0    0    -1
 $EndComp
@@
 Wire Wire Line
 	14000 13750 15700 13750
+$Comp
+L MystiqueJamma-eagle-import:GND #GND0102
+U 1 0 5C2BAFD6
+P 3000 6900
+F 0 "#GND0102" H 3000 6900 50  0001 C CNN
+F 1 "GND" H 2900 6800 59  0000 L BNN
+F 2 "" H 3000 6900 50  0001 C CNN
+F 3 "" H 3000 6900 50  0001 C CNN
+	1    3000 6900
+	1    0    0    -1
+$EndComp
+$Comp
+L MystiqueJamma-eagle-import:+5V #P+0105
+U 1 0 5C37AAB6
+P 4150 6650
+F 0 "#P+0105" H 4150 6650 50  0001 C CNN
+F 1 "+5V" V 4000 6550 59  0000 L BNN
+F 2 "" H 4150 6650 50  0001 C CNN
+F 3 "" H 4150 6650 50  0001 C CNN
+	1    4150 6650
+	0    1    1    0
+$EndComp
+Wire Wire Line
+	4050 6650 3900 6650
+Wire Wire Line
+	3000 6650 3000 6800
+$Comp
+L MystiqueJamma-eagle-import:C4E6-K EVB1
+U 3 0 5CA39EEC
+P 3400 7550
+F 0 "EVB1" H 3250 8580 59  0000 L BNN
+F 1 "C4E6-K" H 3300 8200 59  0000 L BNN
+F 2 "MystiqueJamma:E6V33_BELOW" H 3400 7550 50  0001 C CNN
+F 3 "" H 3400 7550 50  0001 C CNN
+	3    3400 7550
+	1    0    0    -1
+$EndComp
+Wire Wire Line
+	6350 7150 10300 7150
+Wire Wire Line
+	10300 6400 10300 7150
+Wire Wire Line
+	4900 7150 5500 7150
+Text Label 4900 7150 2    50   ~ 0
+VGA_DET_IN
+Wire Wire Line
+	2400 10500 3000 10500
+Text Label 2400 10500 0    50   ~ 0
+VGA_DET_IN
 Wire Bus Line
 	13800 7800 13800 13650

Commit message: Added Micro SD card connector
Parts:
- added J2: Micro_SD_Card, Connector_Card:microSD_HC_Wuerth_693072010801, symbol Connector:Micro_SD_Card
Connections:
- wire segments 775 -> 782
- no-connect marks 46 -> 49
Changed lines of the file:
@@
 Sheet 1 1
 Title "Mystique Jamma"
-Date "2018-12-04"
-Rev "A"
+Date "2018-12-19"
+Rev "B"
 Comp "Reinaldo Flamino / Danjovic"
 Comment1 ""
@@
 Wire Wire Line
 	12000 14250 12200 14250
-Wire Wire Line
-	12000 14250 11100 14250
-Connection ~ 12000 14250
-Text Label 11100 14250 0    50   ~ 0
+Text Label 11050 10350 0    50   ~ 0
 SD_DATAOUT
 Wire Wire Line
@@
 Wire Wire Line
 	11700 14350 11700 14050
-Wire Wire Line
-	11700 14350 11100 14350
-Connection ~ 11700 14350
-Text Label 11100 14350 0    50   ~ 0
+Text Label 11050 9950 0    50   ~ 0
 SD_DATAIN
-Wire Wire Line
-	12200 14450 11100 14450
-Text Label 11100 14450 0    50   ~ 0
+Text Label 11050 10150 0    50   ~ 0
 SD_CNT_SCLK
-Wire Wire Line
-	12200 14550 11100 14550
-Text Label 11100 14550 0    50   ~ 0
+Text Label 11050 9850 0    50   ~ 0
 SD_CS
 Wire Wire Line
@@
 	7500 9900 7600 10000
 Entry Wire Line
-	11000 14150 11100 14250
-Entry Wire Line
-	11000 14250 11100 14350
-Entry Wire Line
-	11000 14350 11100 14450
-Entry Wire Line
-	11000 14450 11100 14550
-Entry Wire Line
 	3500 11200 3600 11300
 Entry Wire Line
@@
 Text Label 2400 10500 0    50   ~ 0
 VGA_DET_IN
+$Comp
+L Connector:Micro_SD_Card J2
+U 1 1 5C270111
+P 12450 10050
+F 0 "J2" H 12400 10767 50  0000 C CNN
+F 1 "Micro_SD_Card" H 12400 10676 50  0000 C CNN
+F 2 "Connector_Card:microSD_HC_Wuerth_693072010801" H 13600 10350 50  0001 C CNN
+F 3 "http://katalog.we-online.de/em/datasheet/693072010801.pdf" H 12450 10050 50  0001 C CNN
+	1    12450 10050
+	1    0    0    -1
+$EndComp
+Wire Wire Line
+	11050 9850 11550 9850
+Wire Wire Line
+	11050 9950 11550 9950
+Wire Wire Line
+	10950 10050 11550 10050
+Wire Wire Line
+	11050 10150 11550 10150
+Wire Wire Line
+	11050 10350 11550 10350
+NoConn ~ 11550 9750
+NoConn ~ 11550 10450
+$Comp
+L MystiqueJamma-eagle-import:GND #GND033
+U 1 0 5C94C078
+P 10950 10550
+F 0 "#GND033" H 10950 10550 50  0001 C CNN
+F 1 "GND" H 10850 10450 59  0000 L BNN
+F 2 "" H 10950 10550 50  0001 C CNN
+F 3 "" H 10950 10550 50  0001 C CNN
+	1    10950 10550
+	1    0    0    -1
+$EndComp
+NoConn ~ 13250 10650
+$Comp
+L MystiqueJamma-eagle-import:+3V3 #+3V09
+U 1 0 5CA1018B
+P 10850 10050
+F 0 "#+3V09" H 10850 10050 50  0001 C CNN
+F 1 "+3V3" V 11000 9950 59  0000 L BNN
+F 2 "" H 10850 10050 50  0001 C CNN
+F 3 "" H 10850 10050 50  0001 C CNN
+	1    10850 10050
+	0    -1   -1   0
+$EndComp
+Wire Wire Line
+	10950 10250 10950 10450
+Wire Wire Line
+	10950 10250 11550 10250
+Text Label 11150 14250 0    50   ~ 0
+SD_DATAOUT
+Text Label 11150 14350 0    50   ~ 0
+SD_DATAIN
+Text Label 11150 14450 0    50   ~ 0
+SD_CNT_SCLK
+Text Label 11150 14550 0    50   ~ 0
+SD_CS
+Entry Wire Line
+	11000 14150 11100 14250
+Entry Wire Line
+	11000 14250 11100 14350
+Entry Wire Line
+	11000 14350 11100 14450
+Entry Wire Line
+	11000 14450 11100 14550
+Wire Wire Line
+	11100 14250 12000 14250
+Connection ~ 12000 14250
+Wire Wire Line
+	11700 14350 11100 14350
+Connection ~ 11700 14350
+Wire Wire Line
+	11100 14450 12200 14450
+Wire Wire Line
+	12200 14550 11100 14550
 Wire Bus Line
 	13800 7800 13800 13650
